File: Hardware/hardware v4 (ble)/hardware v4 pro max(mini patch effectué)/hardware v4 pro max.kicad_pcb (KiCad board)
At the start: 6 copper layers, 26.4 x 19 mm, 78 parts, among them IC1 MLPF-WB-01E3, IC2 W25Q128JVPIQ_TR, J1 SM06B-SRSS-TB, J3 OLED, J4 USB_C_Receptacle_USB2.0_14P, Q1 2N7002K, SW1 Int, SW4 boot, SW5 RSTBTN, U1 STM32WB55CGUx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

Commit message: code
Routing:
- net GND: vias 143 -> 138
Changed lines of the file:
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@@
 	)
 	(via
-		(at 140.09 94.19)
+		(at 140.62 94.22)
 		(size 0.4)
 		(drill 0.3)
@@
 	)
 	(via
-		(at 142.19 91.57)
-		(size 0.4)
-		(drill 0.3)
-		(layers "F.Cu" "B.Cu")
-		(free yes)
-		(net 4)
-	)
-	(via
 		(at 140.14 98.08)
 		(size 0.4)
@@
 	)
 	(via
-		(at 142.17 93.68)
-		(size 0.4)
-		(drill 0.3)
-		(layers "F.Cu" "B.Cu")
-		(free yes)
-		(net 4)
-	)
-	(via
 		(at 144.73 94.04)
 		(size 0.4)
@@
 	)
 	(via
-		(at 138.86 92.44)
-		(size 0.4)
-		(drill 0.3)
-		(layers "F.Cu" "B.Cu")
-		(free yes)
-		(net 4)
-	)
-	(via
 		(at 149.85 106.52)
 		(size 0.4)
@@
 	)
 	(via
-		(at 139.38 94.05)
-		(size 0.4)
-		(drill 0.3)
-		(layers "F.Cu" "B.Cu")
-		(free yes)
-		(net 4)
-	)
-	(via
 		(at 150.87 106.52)
 		(size 0.4)
@@
 	)
 	(via
-		(at 143.44 91.56)
-		(size 0.4)
-		(drill 0.3)
-		(layers "F.Cu" "B.Cu")
-		(free yes)
-		(net 4)
-	)
-	(via
 		(at 131.98 93.3)
 		(size 0.4)
@@
 	)
 	(segment
-		(start 140.9325 103.263437)
-		(end 140.9325 102.8675)
+		(start 142.82 97.14)
+		(end 142.78 97.18)
 		(width 0.2)
 		(layer "F.Cu")
@@
 	)
 	(segment
-		(start 139.4325 103.1875)
-		(end 139.4325 102.8675)
+		(start 141.54 104.051948)
+		(end 141.54 104.09)
 		(width 0.2)
 		(layer "F.Cu")
@@
 	)
 	(segment
-		(start 142.12 97.18)
-		(end 142.69 97.18)
+		(start 139.4325 103.1875)
+		(end 139.4325 102.8675)
 		(width 0.2)
 		(layer "F.Cu")
@@
 	)
 	(segment
-		(start 142.66 97.68)
-		(end 142.72 97.62)
+		(start 142.78 97.18)
+		(end 142.12 97.18)
 		(width 0.2)
 		(layer "F.Cu")
@@
 	)
 	(segment
-		(start 141.02449 103.355427)
-		(end 141.54 103.870937)
+		(start 141.034026 103.545974)
+		(end 141.54 104.051948)
 		(width 0.2)
 		(layer "F.Cu")
@@
 	)
 	(segment
-		(start 142.69 97.18)
-		(end 142.71 97.16)
+		(start 141.034026 103.545974)
+		(end 140.9325 103.444448)
 		(width 0.2)
 		(layer "F.Cu")
@@
 	)
 	(segment
-		(start 141.02449 103.355427)
-		(end 140.9325 103.263437)
+		(start 142.81 97.68)
+		(end 142.12 97.68)
 		(width 0.2)
 		(layer "F.Cu")
@@
 	)
 	(segment
-		(start 142.12 97.68)
-		(end 142.66 97.68)
+		(start 140.9325 103.444448)
+		(end 140.9325 102.8675)
 		(width 0.2)
 		(layer "F.Cu")
@@
 	)
 	(segment
-		(start 141.54 103.870937)
-		(end 141.54 104.09)
+		(start 142.82 97.69)
+		(end 142.81 97.68)
 		(width 0.2)
 		(layer "F.Cu")
@@
 	)
 	(via
-		(at 142.71 97.16)
+		(at 142.82 97.14)
 		(size 0.4)
 		(drill 0.3)
@@
 	)
 	(via
-		(at 141.02449 103.355427)
+		(at 141.034026 103.545974)
 		(size 0.4)
 		(drill 0.3)
@@
 	)
 	(via
-		(at 142.72 97.62)
+		(at 142.82 97.69)
 		(size 0.4)
 		(drill 0.3)
@@
 	)
 	(segment
-		(start 141.92 102.21)
-		(end 141.92 102.459917)
+		(start 139.3 103.32)
+		(end 139.3 102.1)
 		(width 0.2)
 		(layer "B.Cu")
@@
 	)
 	(segment
-		(start 139.3 103.32)
-		(end 139.3 102.1)
+		(start 142.82 97.69)
+		(end 142.82 98.936)
 		(width 0.2)
 		(layer "B.Cu")
@@
 	)
 	(segment
-		(start 142.72 97.62)
-		(end 142.72 99.036)
-		(width 0.2)
-		(layer "B.Cu")
-		(net 5)
-	)
-	(segment
 		(start 133.21 94.09)
 		(end 133.29 94.01)
@@
 	)
 	(segment
-		(start 141.92 102.459917)
-		(end 141.02449 103.355427)
+		(start 139.3 102.1)
+		(end 139.35 102.05)
 		(width 0.2)
 		(layer "B.Cu")
@@
 	)
 	(segment
-		(start 139.3 102.1)
-		(end 139.35 102.05)
+		(start 141.034026 103.545974)
+		(end 141.92 102.66)
 		(width 0.2)
 		(layer "B.Cu")
@@
 	)
 	(segment
-		(start 142.72 99.036)
-		(end 142.463 99.293)
+		(start 139.89 96.68)
+		(end 140.21 97)
 		(width 0.2)
 		(layer "B.Cu")
@@
 	)
 	(segment
-		(start 139.89 96.68)
-		(end 140.21 97)
+		(start 141.92 102.66)
+		(end 141.92 102.21)
 		(width 0.2)
 		(layer "B.Cu")
@@
 	)
 	(segment
+		(start 142.82 98.936)
+		(end 142.463 99.293)
+		(width 0.2)
+		(layer "B.Cu")
+		(net 5)
+	)
+	(segment
 		(start 150.625 100.33)
 		(end 150.595 100.36)
@@
 	)
 	(via
-		(at 140.941084 103.890141)
+		(at 140.96 104.049671)
 		(size 0.4)
 		(drill 0.3)
@@
 	)
 	(segment
-		(start 141.22019 103.890141)
-		(end 141.42 103.690331)
+		(start 141.42 103.690331)
+		(end 141.42 102.53)
 		(width 0.15)
 		(layer "In3.Cu")
@@
 	)
 	(segment
-		(start 141.42 103.690331)
-		(end 141.42 102.53)
+		(start 142.335 95.735)
+		(end 142.9 95.17)
 		(width 0.15)
 		(layer "In3.Cu")
@@
 	)
 	(segment
-		(start 140.941084 103.890141)
-		(end 141.22019 103.890141)
+		(start 141.06066 104.049671)
+		(end 141.42 103.690331)
 		(width 0.15)
 		(layer "In3.Cu")
@@
 	)
 	(segment
-		(start 142.335 95.735)
-		(end 142.9 95.17)
+		(start 140.96 104.049671)
+		(end 141.06066 104.049671)
 		(width 0.15)
 		(layer "In3.Cu")
@@
 	)
 	(segment
-		(start 140.941084 105.141916)
-		(end 140.91 105.173)
+		(start 140.96 104.049671)
+		(end 140.96 105.123)
 		(width 0.15)
 		(layer "B.Cu")
@@
 	)
 	(segment
-		(start 140.941084 103.890141)
-		(end 140.941084 105.141916)
+		(start 140.96 105.123)
+		(end 140.91 105.173)
 		(width 0.15)
 		(layer "B.Cu")
@@
 	)
 	(segment
-		(start 141.4325 95.500767)
-		(end 141.54 95.393267)
+		(start 141.4325 95.56612)
+		(end 141.4325 95.9925)
 		(width 0.2)
 		(layer "F.Cu")
@@
 	)
 	(segment
-		(start 141.4325 95.9925)
-		(end 141.4325 95.500767)
+		(start 141.622851 95.375769)
+		(end 141.4325 95.56612)
 		(width 0.2)
 		(layer "F.Cu")
@@
 	)
 	(via
-		(at 141.54 95.393267)
+		(at 141.622851 95.375769)
 		(size 0.4)
 		(drill 0.3)
@@
 	)
 	(segment
-		(start 141.34 95.593267)
-		(end 141.34 97.095736)
+		(start 144.474264 100.23)
+		(end 149.775 100.23)
 		(width 0.2)
 		(layer "In2.Cu")
@@
 	)
 	(segment
-		(start 141.54 95.393267)
-		(end 141.34 95.593267)
+		(start 141.622851 95.375769)
+		(end 141.34 95.65862)
 		(width 0.2)
 		(layer "In2.Cu")
@@
 	)
 	(segment
-		(start 149.775 100.23)
-		(end 150.595 99.41)
+		(start 141.34 97.095736)
+		(end 144.474264 100.23)
 		(width 0.2)
 		(layer "In2.Cu")
@@
 	)
 	(segment
-		(start 144.474264 100.23)
-		(end 149.775 100.23)
+		(start 141.34 95.65862)
+		(end 141.34 97.095736)
 		(width 0.2)
 		(layer "In2.Cu")
@@
 	)
 	(segment
-		(start 141.34 97.095736)
-		(end 144.474264 100.23)
+		(start 149.775 100.23)
+		(end 150.595 99.41)
 		(width 0.2)
 		(layer "In2.Cu")
@@
 	)
 	(zone
+		(net 0)
+		(net_name "")
+		(layer "F.Cu")
+		(hatch edge 0.5)
+		(connect_pads
+			(clearance 0)
+		)
+		(min_thickness 0.25)
+		(filled_areas_thickness no)
+		(keepout
+			(tracks allowed)
+			(vias allowed)
+			(pads allowed)
+			(copperpour not_allowed)
+			(footprints allowed)
+		)
+		(fill
+			(thermal_gap 0.5)
+			(thermal_bridge_width 0.5)
+		)
+		(polygon
+			(pts
+				(xy 134.09 91.07) (xy 134.09 92.9) (xy 138.46 92.9) (xy 138.51 92.85) (xy 138.51 91.04) (xy 134.12 91.04)
+			)
+		)
+	)
+	(zone
 		(net 5)
 		(net_name "+3.3V")
@@
 			)
 		)
+	)
+	(zone
+		(net 0)
+		(net_name "")
+		(layer "F.Cu")
+		(hatch edge 0.5)
+		(connect_pads
+			(clearance 0)
+		)
+		(min_thickness 0.25)
+		(filled_areas_thickness no)
+		(keepout
+			(tracks allowed)
+			(vias allowed)
+			(pads allowed)
+			(copperpour not_allowed)
+			(footprints allowed)
+		)
+		(fill
+			(thermal_gap 0.5)
+			(thermal_bridge_width 0.5)
+		)
+		(polygon
+			(pts
+				(xy 141.69 96.95) (xy 141.69 98.37) (xy 141.74 98.42) (xy 142.7 98.42) (xy 142.73 98.45) (xy 142.73 99.46)
+				(xy 142.77 99.5) (xy 146.28 99.5) (xy 146.28 96.98) (xy 146.25 96.95)
+			)
+		)
