File: Hardware/hardware v8/hardware v8/BTN_CONN.kicad_sch (KiCad schematic)
At the start: 15 parts, among them J3 OLED, J4 USB_C_Receptacle_USB2.0_14P

Commit message: v8
Parts:
- removed J4: USB_C_Receptacle_USB2.0_14P, samacsys:USB4110GFA, symbol Vraielogousbcwurth:USB_C_Receptacle_USB2.0_14P
- removed R14, R15: 5.1k, Resistor_SMD:R_0201_0603Metric_Pad0.64x0.40mm_HandSolder, symbol Device:R_Small
- added C14: 100n, Capacitor_SMD:C_0201_0603Metric_Pad0.64x0.40mm_HandSolder, symbol Device:C_Small
- added J1: USB4720-03-A, samacsys2:USB472003A, symbol samacsys2:USB4720-03-A
- added R19, R3: 470k, Resistor_SMD:R_0201_0603Metric_Pad0.64x0.40mm_HandSolder, symbol Device:R_Small
- added R22, R23: 5.1k, Resistor_SMD:R_0201_0603Metric_Pad0.64x0.40mm_HandSolder, symbol Device:R_Small
Connections:
- net BAT- is gone; now on net GND: U5.1
- net +3.3V: no longer J3.2 (Pin_2)
- net D+: now also J1.A6 (DP1), J1.B6 (DP2)
- net D-: now also J1.A7 (DN1), J1.B7 (DN2)
- net GND: now also C14.2, J1.A1 (GND_1), J1.A12 (GND_2), J1.MH1, J1.MH2, J1.MH3, J1.MH4, J1.MH5, J1.MH6, R19.1, R22.2, R23.2
- net vusb: now also J1.A4 (VBUS_1), J1.A9 (VBUS_2), R3.2
- new net: J1.A5 (CC1), R22.1
- new net: J1.B5 (CC2), R23.1
- new net 3.3V_AUX: J3.2 (Pin_2)
- new net USB_DETECT: C14.1, R19.2, R3.1
Other:
- moved on the sheet: D2, J3, U5

Commit message: up
Parts:
- removed D2: 82400274, samacsys:SOT65P210X110-6N, symbol samacsys:82400274
- added D1, D2: PESD5V0S1UL-QYL, samacsys2:PESD5V0S1ULQYL, symbol samacsys2:PESD5V0S1UL-QYL
- S3: footprint samacsys:PTS845VM20PSMTR4LFS -> samacsys2:PTS845VM20PSMTR4LFS
Connections:
- net D+: now also D1.1 (K)
- net D-: now also D2.2 (A)
- net GND: now also D1.2 (A), D2.1 (K)
- no-connect marks 4 -> 2
Other:
- note added: "BAT"
- note removed: "ESD PROTECTION"
- moved on the sheet: C14, J1, J3, R19, R22, R23, R3

Commit message: up
Parts:
- added J2: 503548-0622, samacsys2:5035480622, symbol samacsys2:503548-0622
Connections:
- net 3.3V_AUX: now also J2.1, J2.6
- net GND: now also J2.10, J2.3, J2.4, J2.7, J2.8, J2.9
- net OLED_SCL: now also J2.5
- net OLED_SDA: now also J2.2
Other:
- note added: "AUX"
- moved on the sheet: U5

Commit message: up
Parts:
- J3: now not fitted
- R7, R8, R9: value 10k -> 20k
Changed lines of the file:
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@@
 			)
 		)
-		(property "Value" "10k"
+		(property "Value" "20k"
 			(at 236.22 109.2199 0)
 			(effects
@@
 			)
 		)
-		(property "Value" "10k"
+		(property "Value" "20k"
 			(at 236.22 137.1599 0)
 			(effects
@@
 			)
 		)
-		(property "Value" "10k"
+		(property "Value" "20k"
 			(at 237.49 82.5499 0)
 			(effects
@@
 		(in_bom yes)
 		(on_board yes)
-		(dnp no)
+		(dnp yes)
 		(fields_autoplaced yes)
 		(property "Reference" "J3"

Commit message: up
Parts:
- R19, R3: Mouser Part Number (none) -> 603-AC0201FR-07470KL; Mouser Price/Stock (none) -> https://www.mouser.fr/ProductDetail/YAGEO/AC0201FR-07470KL?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
- R22, R23: Mouser Part Number (none) -> 603-AF0201FR-075K1L; Mouser Price/Stock (none) -> https://www.mouser.fr/ProductDetail/YAGEO/AF0201FR-075K1L?q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
- R7, R8, R9: Mouser Part Number (none) -> 603-AC0201FR-0720KL; Mouser Price/Stock (none) -> https://www.mouser.fr/ProductDetail/YAGEO/AC0201FR-0720KL?q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
- U5: Mouser Part Number (none) -> 306-BM02BSRSSTBLFSNP; Mouser Price/Stock (none) -> https://www.mouser.fr/ProductDetail/JST-Commercial/BM02B-SR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
Changed lines of the file:
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@@
 			)
 		)
+		(property "Mouser Part Number" "603-AC0201FR-07470KL"
+			(at 135.89 46.99 90)
+			(effects
+				(font
+					(size 1.27 1.27)
+				)
+				(hide yes)
+			)
+		)
+		(property "Mouser Price/Stock" "https://www.mouser.fr/ProductDetail/YAGEO/AC0201FR-07470KL?qs=NgbZBzc1CyH0J6cte9SzFw%3D%3D"
+			(at 135.89 46.99 90)
+			(effects
+				(font
+					(size 1.27 1.27)
+				)
+				(hide yes)
+			)
+		)
 		(pin "2"
 		)
@@
 			)
 		)
+		(property "Mouser Part Number" "603-AC0201FR-0720KL"
+			(at 233.68 107.95 0)
+			(effects
+				(font
+					(size 1.27 1.27)
+				)
+				(hide yes)
+			)
+		)
+		(property "Mouser Price/Stock" "https://www.mouser.fr/ProductDetail/YAGEO/AC0201FR-0720KL?qs=NgbZBzc1CyEbaKDOC3%252BFfg%3D%3D"
+			(at 233.68 107.95 0)
+			(effects
+				(font
+					(size 1.27 1.27)
+				)
+				(hide yes)
+			)
+		)
 		(pin "2"
 		)
@@
 			)
 		)
+		(property "Mouser Part Number" "603-AC0201FR-0720KL"
+			(at 233.68 135.89 0)
+			(effects
+				(font
+					(size 1.27 1.27)
+				)
+				(hide yes)
+			)
+		)
+		(property "Mouser Price/Stock" "https://www.mouser.fr/ProductDetail/YAGEO/AC0201FR-0720KL?qs=NgbZBzc1CyEbaKDOC3%252BFfg%3D%3D"
+			(at 233.68 135.89 0)
+			(effects
+				(font
+					(size 1.27 1.27)
+				)
+				(hide yes)
+			)
+		)
 		(pin "2"
 		)
@@
 			)
 		)
+		(property "Mouser Part Number" "603-AC0201FR-0720KL"
+			(at 234.95 81.28 0)
+			(effects
+				(font
+					(size 1.27 1.27)
+				)
+				(hide yes)
+			)
+		)
+		(property "Mouser Price/Stock" "https://www.mouser.fr/ProductDetail/YAGEO/AC0201FR-0720KL?qs=NgbZBzc1CyEbaKDOC3%252BFfg%3D%3D"
+			(at 234.95 81.28 0)
+			(effects
+				(font
+					(size 1.27 1.27)
+				)
+				(hide yes)
+			)
+		)
 		(pin "2"
 		)
@@
 			)
 		)
+		(property "Mouser Part Number" "603-AF0201FR-075K1L"
+			(at 41.91 46.99 90)
+			(effects
+				(font
+					(size 1.27 1.27)
+				)
+				(hide yes)
+			)
+		)
+		(property "Mouser Price/Stock" "https://www.mouser.fr/ProductDetail/YAGEO/AF0201FR-075K1L?qs=tggtontpCXOBTGA3imPYYA%3D%3D"
+			(at 41.91 46.99 90)
+			(effects
+				(font
+					(size 1.27 1.27)
+				)
+				(hide yes)
+			)
+		)
 		(pin "2"
 		)
@@
 			)
 		)
+		(property "Mouser Part Number" "603-AC0201FR-07470KL"
+			(at 135.89 57.15 90)
+			(effects
+				(font
+					(size 1.27 1.27)
+				)
+				(hide yes)
+			)
+		)
+		(property "Mouser Price/Stock" "https://www.mouser.fr/ProductDetail/YAGEO/AC0201FR-07470KL?qs=NgbZBzc1CyH0J6cte9SzFw%3D%3D"
+			(at 135.89 57.15 90)
+			(effects
+				(font
+					(size 1.27 1.27)
+				)
+				(hide yes)
+			)
+		)
 		(pin "2"
 		)
@@
 			)
 		)
+		(property "Mouser Part Number" "603-AF0201FR-075K1L"
+			(at 41.91 62.23 90)
+			(effects
+				(font
+					(size 1.27 1.27)
+				)
+				(hide yes)
+			)
+		)
+		(property "Mouser Price/Stock" "https://www.mouser.fr/ProductDetail/YAGEO/AF0201FR-075K1L?qs=tggtontpCXOBTGA3imPYYA%3D%3D"
+			(at 41.91 62.23 90)
+			(effects
+				(font
+					(size 1.27 1.27)
+				)
+				(hide yes)
+			)
+		)
 		(pin "2"
 		)
@@
 			(at 99.06 114.3 0)
 			(effects
+				(font
+					(size 1.27 1.27)
+				)
+				(hide yes)
+			)
+		)
+		(property "Mouser Part Number" "306-BM02BSRSSTBLFSNP"
+			(at 99.06 114.3 0)
+			(effects
+				(font
+					(size 1.27 1.27)
+				)
+				(hide yes)
+			)
+		)
+		(property "Mouser Price/Stock" "https://www.mouser.fr/ProductDetail/JST-Commercial/BM02B-SRSS-TBLFSN?qs=sGAEpiMZZMvlX3nhDDO4AFC8wiFPNfngi093wynrZHM%3D"
+			(at 99.06 114.3 0)
+			(effects
