File: Hardware/hardware v8/hardware v8/hardware_V8.kicad_pcb (KiCad board)
At the start: 6 copper layers, 21 x 19 mm, 33 parts, among them IC1 MLPF-WB-01E3, IC4 MAX-M10S-00B, J3 OLED, J4 USB_C_Receptacle_USB2.0_14P, U4 USBLC6-2SC6

Commit message: v8
Parts:
- removed ANT1: 74889302450, antennesmd:74889302450
- removed C9: 0.1u, Capacitor_SMD:C_0402_1005Metric
- removed FL1: LFCN-2400D, LFCN2400D:DLF162500LT5028A1
- removed the J3 at (148.6, 93.0)
- removed the J3 at (99.2, 98.8)
- removed J4: USB_C_Receptacle_USB2.0_14P, USBCWURTH:USBC-WURTH
- removed R14 (x2), R15 (x2): 5.1k, Resistor_SMD:R_0402_1005Metric
- removed the S2 at (142.0, 108.3)
- removed the S2 at (136.1, 108.3)
- removed the S2 at (136.6, 92.8)
- removed U4: USBLC6-2SC6, Package_TO_SOT_SMD:SOT-23-6
- added C1: 1u, Capacitor_SMD:C_0402_1005Metric, F.Cu at (127.7, 91.8)
- added C13: 100n, Capacitor_SMD:C_0201_0603Metric_Pad0.64x0.40mm_HandSolder, F.Cu at (123.8, 101.0)
- added C15: 10n, Capacitor_SMD:C_0201_0603Metric_Pad0.64x0.40mm_HandSolder, B.Cu at (129.7, 96.3)
- added C16: 1u, Capacitor_SMD:C_0402_1005Metric, B.Cu at (129.7, 97.2)
- added C18: 100n, Capacitor_SMD:C_0201_0603Metric_Pad0.64x0.40mm_HandSolder, F.Cu at (123.8, 102.5)
- added C25: 100n, Capacitor_SMD:C_0201_0603Metric_Pad0.64x0.40mm_HandSolder, F.Cu at (122.6, 90.8)
- added C26: 100n, Capacitor_SMD:C_0201_0603Metric_Pad0.64x0.40mm_HandSolder, B.Cu at (129.7, 91.8)
- added C27: 100n, Capacitor_SMD:C_0201_0603Metric_Pad0.64x0.40mm_HandSolder, B.Cu at (129.7, 98.1)
- added C28: 4.7u, Capacitor_SMD:C_0402_1005Metric, B.Cu at (129.7, 92.7)
- added C29: 1u, Capacitor_SMD:C_0402_1005Metric, F.Cu at (118.6, 104.7)
- added C4: 1u, Capacitor_SMD:C_0402_1005Metric, F.Cu at (131.4, 91.9)
- added C5: 1u, Capacitor_SMD:C_0402_1005Metric, F.Cu at (127.7, 93.6)
- added IC5: LTC4065EDC#TRMPBF, samacsys2:SON50P200X200X80-7N-D, F.Cu at (117.0, 106.5)
- added IC6: W25Q128JVPIQ, samacsys2:SON127P600X500X80-9N-D, F.Cu at (128.2, 97.3)
- added J1: USB4720-03-A, samacsys2:USB472003A, B.Cu at (113.0, 97.7)
- added J3: OLED, Connector_PinSocket_2.54mm:PinSocket_1x04_P2.54mm_Vertical, B.Cu at (126.2, 89.6)
- added LEDBLUE1: 150040BS73240, LED_SMD:LED_0402_1005Metric, F.Cu at (113.2, 88.0)
- added LEDGREEN1: 150040GS73240, LED_SMD:LED_0402_1005Metric, F.Cu at (115.6, 88.0)
- added LEDRED1: 150040RS73240, LED_SMD:LED_0402_1005Metric, F.Cu at (112.3, 105.9)
- added R1: 510R, Resistor_SMD:R_0201_0603Metric_Pad0.64x0.40mm_HandSolder, F.Cu at (115.8, 89.9)
- added R10: 470k, Resistor_SMD:R_0201_0603Metric_Pad0.64x0.40mm_HandSolder, B.Cu at (129.7, 93.8)
- added R16: 470k, Resistor_SMD:R_0201_0603Metric_Pad0.64x0.40mm_HandSolder, B.Cu at (129.7, 94.5)
- added R17: 20k, Resistor_SMD:R_0201_0603Metric_Pad0.64x0.40mm_HandSolder, F.Cu at (114.5, 107.4)
- added R18: 10k, Resistor_SMD:R_0201_0603Metric_Pad0.64x0.40mm_HandSolder, F.Cu at (130.9, 93.2)
- added R2: 510R, Resistor_SMD:R_0201_0603Metric_Pad0.64x0.40mm_HandSolder, F.Cu at (113.0, 89.9)
- added R21: 10k, Resistor_SMD:R_0201_0603Metric_Pad0.64x0.40mm_HandSolder, F.Cu at (125.7, 91.1)
- added R22: 5.1k, Resistor_SMD:R_0201_0603Metric_Pad0.64x0.40mm_HandSolder, F.Cu at (117.8, 100.1)
- added R3: 470k, Resistor_SMD:R_0201_0603Metric_Pad0.64x0.40mm_HandSolder, F.Cu at (119.3, 103.8)
- added R4: 510R, Resistor_SMD:R_0201_0603Metric_Pad0.64x0.40mm_HandSolder, F.Cu at (114.9, 104.3)
- added R5: 10k, Resistor_SMD:R_0201_0603Metric_Pad0.64x0.40mm_HandSolder, F.Cu at (129.2, 94.2)
- added R6: 10k, Resistor_SMD:R_0201_0603Metric_Pad0.64x0.40mm_HandSolder, F.Cu at (123.8, 101.8)
- added S1: PTS845VM20PSMTR4_LFS, samacsys:PTS845VM20PSMTR4LFS, B.Cu at (114.3, 106.3)
- added S2: PTS845VM20PSMTR4_LFS, samacsys:PTS845VM20PSMTR4LFS, B.Cu at (119.8, 106.3)
- added S3: PTS845VM20PSMTR4_LFS, samacsys:PTS845VM20PSMTR4LFS, B.Cu at (114.4, 89.1)
- added SW4: boot, samacsys:KXT341LHS, F.Cu at (120.7, 102.0)
- added TP3: SWCLK, samacsys:pad_0.7mm, B.Cu at (131.3, 97.4)
- added TP4: SWDIO, samacsys:pad_0.7mm, B.Cu at (131.3, 96.1)
- added TP5: NRST, samacsys:pad_0.7mm, B.Cu at (131.3, 98.7)
- added TP6: GND, samacsys:pad_0.7mm, B.Cu at (131.3, 94.8)
- added U1: STM32L432KCUx, Package_DFN_QFN:QFN-32-1EP_5x5mm_P0.5mm_EP3.45x3.45mm, F.Cu at (121.3, 97.4)
- added U2: ldln025pu, samacsys:ldln025pu, F.Cu at (128.9, 93.1)
- added U5: ~, Connector_JST:JST_SH_BM02B-SRSS-TB_1x02-1MP_P1.00mm_Vertical, F.Cu at (129.6, 89.8)
- C10: value 1u -> 100n; footprint Capacitor_SMD:C_0402_1005Metric -> Capacitor_SMD:C_0201_0603Metric_Pad0.64x0.40mm_HandSolder
- C11, C14: footprint Capacitor_SMD:C_0402_1005Metric -> Capacitor_SMD:C_0201_0603Metric_Pad0.64x0.40mm_HandSolder
- C19: value 100n -> 4.7u
- C20, C6, C7: value 10n -> 100n; footprint Capacitor_SMD:C_0402_1005Metric -> Capacitor_SMD:C_0201_0603Metric_Pad0.64x0.40mm_HandSolder
- C8: value 1u -> 100n; footprint Capacitor_SMD:C_0402_1005Metric -> Capacitor_SMD:C_0201_0603Metric_Pad0.64x0.40mm_HandSolder; moved to B.Cu
- IC1: value MLPF-WB-01E3 -> TPS22960RSER; footprint MLPFWB01E3:MLPFWB01E3 -> samacsys2:TPS22960RSER
- R11, R12: value 470R -> 510R; footprint Resistor_SMD:R_0402_1005Metric -> Resistor_SMD:R_0201_0603Metric_Pad0.64x0.40mm_HandSolder
- R13, R7, R8, R9: footprint Resistor_SMD:R_0402_1005Metric -> Resistor_SMD:R_0201_0603Metric_Pad0.64x0.40mm_HandSolder
- R19: value 10R -> 470k; footprint Resistor_SMD:R_0402_1005Metric -> Resistor_SMD:R_0201_0603Metric_Pad0.64x0.40mm_HandSolder
- R20: value 2.2k -> 10k; footprint Resistor_SMD:R_0402_1005Metric -> Resistor_SMD:R_0201_0603Metric_Pad0.64x0.40mm_HandSolder
- R23: value 2.2k -> 5.1k; footprint Resistor_SMD:R_0402_1005Metric -> Resistor_SMD:R_0201_0603Metric_Pad0.64x0.40mm_HandSolder
- moved R13 21.7 mm to (129.0, 100.5), turned to 180 degrees
- moved C8 19.2 mm to (129.7, 95.2)
- moved IC1 18.7 mm to (126.1, 92.7), turned to -90 degrees
- moved R8 18.7 mm to (120.3, 106.2), turned to -90 degrees
- moved R19 18.3 mm to (121.1, 104.5), turned to 180 degrees
- moved IC4 16.7 mm to (123.4, 97.5), turned to 90 degrees
- moved C6 16.0 mm to (119.2, 106.2), turned to -90 degrees
- moved C11 16.0 mm to (125.7, 100.6), turned to 180 degrees
- moved R9 15.9 mm to (113.8, 89.9), turned to 90 degrees
- moved C14 14.8 mm to (121.1, 103.8)
- moved C20 14.7 mm to (115.0, 89.9), turned to 90 degrees
- moved R20 14.1 mm to (126.2, 94.1)
- moved R11 14.0 mm to (122.1, 92.6)
- moved R7 13.9 mm to (113.8, 106.1), turned to -90 degrees
- moved R12 12.1 mm to (122.1, 91.9)
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Connections:
- C10 pad 1: +3.3V -> GND
- C10 pad 2: Net-(BT1--) -> +3.3V
- C11 pad 1: +3.3V -> 3.3V_AUX
- C14 pad 1: Net-(U5-VDD) -> /USB_DETECT
- C19 pad 1: Net-(U5-VDD) -> GND
- C19 pad 2: GND -> +3.3V
- C20 pad 1: B2 -> /B_PW
- C6 pad 1: B2 -> /B2
- C7 pad 1: B1 -> /B1
- C8 pad 2: Net-(BT1--) -> GND
- IC4 pad 2: unconnected-(IC4-TXD-Pad2) -> Net-(IC4-TXD)
- IC4 pad 3: unconnected-(IC4-RXD-Pad3) -> Net-(IC4-RXD)
- IC4 pad 4: unconnected-(IC4-TIMEPULSE-Pad4) -> /Peripherial/GPS_TP
- IC4 pad 5: unconnected-(IC4-EXTINT-Pad5) -> /Peripherial/GPS_EXT
- IC4 pad 7: unconnected-(IC4-V_IO-Pad7) -> 3.3V_GPS
- IC4 pad 8: unconnected-(IC4-VCC-Pad8) -> 3.3V_GPS
- R11 pad 1: unconnected-(R11-Pad1) -> Net-(IC4-TXD)
- R11 pad 2: /Peripherial/GPS_TX -> /GPS_TX
- R12 pad 1: /Peripherial/GPS_RX -> Net-(IC4-RXD)
- R12 pad 2: unconnected-(R12-Pad2) -> /GPS_RX
- R13 pad 1: /Peripherial/SPI_CS -> /SPI_CS
- R13 pad 2: +3.3V -> 3.3V_AUX
- R19 pad 1: +3.3V -> GND
- R19 pad 2: Net-(U5-VDD) -> /USB_DETECT
- R20 pad 1: +3.3V -> GND
- R20 pad 2: /Peripherial/COMPAS_SCL -> /GPS_EN
- R23 pad 1: /Peripherial/COMPAS_SDA -> Net-(J1-CC2)
- R23 pad 2: +3.3V -> GND
- R7 pad 1: +3.3V -> /B1
- R7 pad 2: B1 -> +3.3V
- R8 pad 1: +3.3V -> /B2
- R8 pad 2: B2 -> +3.3V
- R9 pad 1: +3.3V -> /B_PW
- R9 pad 2: B2 -> +3.3V
Routing:
- net BAT+: track 0.99 -> 24.9 mm, vias 0 -> 3
- net /SPI_MISO: track 0.00 -> 20.6 mm, vias 0 -> 2
- net /SWDIO: track 0.00 -> 17.3 mm, vias 0 -> 2
- net /SPI_CS: track 0.00 -> 17.3 mm, vias 0 -> 2
- net Net-(U1-PB6): track 0.00 -> 16.9 mm, vias 0 -> 2
- net /SWCLK: track 0.00 -> 16.4 mm, vias 0 -> 2
- net Net-(U1-PB5): track 0.00 -> 14.4 mm, vias 0 -> 2
- net /B_PW: track 0.00 -> 11.1 mm, vias 0 -> 2
- net /B1: track 0.00 -> 11.1 mm, vias 0 -> 2
- net +3.3V: track 0.00 -> 11.0 mm, vias 0 -> 9
- net Net-(IC5-~{CHRG}): track 0.00 -> 9.72 mm, vias 0 -> 2
- net /OLED_SDA: track 0.00 -> 9.44 mm, vias 0 -> 2
- net /OLED_SCL: track 0.00 -> 9.35 mm, vias 0 -> 2
- net /AUX_EN: track 0.00 -> 8.60 mm, vias 0 -> 2
- net /NRST: track 0.00 -> 8.30 mm, vias 0 -> 2
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- added copper zone on B.Cu, net +3.3V
- added copper zone on F.Cu, net +3.3V
- added copper zone on In3.Cu, net +3.3V
- added copper zone on F.Cu, net 3.3V_AUX
- added copper zone on In3.Cu, net 3.3V_AUX
- added copper zone on B.Cu, net 3.3V_GPS
- added copper zone on F.Cu, net 3.3V_GPS
- added copper zone on F.Cu, net BAT+
- added copper zone on In4.Cu, net GND
- added copper zone on F.Cu, net Net-(U1-PH3)
- added copper zone on F.Cu, net vusb
- added copper zone on In3.Cu, net vusb
- removed copper zone on In4.Cu, net +3.3V
- removed copper zone on In2.Cu, net GND
- removed copper zone on In3.Cu, net GND
Other:
- board size 21 x 19 mm -> 20.5 x 20.8 mm
- board text removed: "mathieu.p"
- board text removed: "pressure"
- board text removed: "swclk"
- board text removed: "swdio"
- board text removed: "swo"

Commit message: up
Parts:
- added D1: PESD5V0S1UL-QYL, samacsys2:PESD5V0S1ULQYL, F.Cu at (117.9, 95.0)
- added D2: PESD5V0S1UL-QYL, samacsys2:PESD5V0S1ULQYL, F.Cu at (117.9, 100.1)
- R20, R21: value 10k -> 100k
- S3: footprint samacsys:PTS845VM20PSMTR4LFS -> samacsys2:PTS845VM20PSMTR4LFS
- moved R22 4.30 mm to (114.9, 103.3)
- moved R23 4.03 mm to (114.9, 92.1)
- moved LEDRED1 1.50 mm to (113.0, 104.5), turned to 0 degrees
- moved R4 0.25 mm to (114.8, 104.5)
- moved R21 0.10 mm to (125.7, 91.2)
- moved LEDBLUE1 0.06 mm to (113.2, 88.0)
Connections:
- C25 pad 1: unconnected-(C25-Pad1) -> Net-(IC4-V_BCKP)
- C8 pad 1: Net-(U1-PA0) -> /ADC_BAT
- IC4 pad 5: /Peripherial/GPS_EXT -> /GPS_EXTINT
- IC4 pad 6: unconnected-(C25-Pad1) -> Net-(IC4-V_BCKP)
- R10 pad 2: Net-(U1-PA0) -> /ADC_BAT
- R16 pad 2: Net-(U1-PA0) -> /ADC_BAT
- U1 pad 14: /B_PW -> /ADC_BAT
- U1 pad 18: unconnected-(U1-PA8-Pad18) -> /GPS_EXTINT
- U1 pad 6: Net-(U1-PA0) -> /B_PW
Routing:
- net /ADC_BAT: track 0.00 -> 11.7 mm, vias 0 -> 1
- net GND: track 0.00 -> 8.35 mm, vias 45 -> 118
- net Net-(U1-PA0): track 7.60 -> 0.00 mm, vias 1 -> 0
- net /GPS_EXTINT: track 0.00 -> 7.11 mm, vias 0 -> 1
- net Net-(J1-CC1): track 1.21 -> 7.38 mm
- net Net-(J1-CC2): track 1.00 -> 6.51 mm
- net /B_PW: track 11.1 -> 15.6 mm
- net unconnected-(C25-Pad1): track 3.85 -> 0.00 mm, vias 1 -> 0
- net Net-(IC4-V_BCKP): track 0.00 -> 3.85 mm, vias 0 -> 1
- net +3.3V: track 11.0 -> 7.30 mm
- net /SPI_MISO: track 20.6 -> 18.3 mm
- net /AUX_EN: track 8.60 -> 6.57 mm
- net /D+: track 2.48 -> 4.42 mm
- net Net-(LEDRED1-A): track 2.65 -> 1.01 mm
- net /D-: track 3.01 -> 4.65 mm
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- added copper zone on In2.Cu, net GND

Commit message: up
Parts:
- added C2: TBD, Capacitor_SMD:C_0402_1005Metric, B.Cu at (126.3, 104.3)
- added C3: TBD, Capacitor_SMD:C_0402_1005Metric, B.Cu at (127.9, 106.7)
- added G***: LOGO, stormtrooper:rex, F.Cu at (125.5, 104.5)
- added J2: 503548-0622, samacsys2:5035480622, B.Cu at (130.5, 89.5)
- added L1: TBD, Inductor_SMD:L_0402_1005Metric, B.Cu at (126.7, 105.8)
- added U3: 146235-0001, samacsys2:146235-0001, B.Cu at (131.4, 104.3)
- moved R13 1.59 mm to (127.5, 100.5)
Connections:
- IC4 pad 11: unconnected-(IC4-RF_IN-Pad11) -> Net-(IC4-RF_IN)
Routing:
- net /OLED_SDA: track 9.40 -> 22.9 mm, vias 2 -> 3
- net /OLED_SCL: track 9.35 -> 20.5 mm, vias 2 -> 3
- net 3.3V_AUX: track 5.73 -> 10.3 mm, vias 2 -> 3
- net Net-(C3-Pad1): track 0.00 -> 3.69 mm
- net Net-(IC4-RF_IN): track 0.00 -> 3.06 mm
- net /SPI_CS: track 16.9 -> 18.8 mm, vias 2 -> 3
- net GND: vias 118 -> 133
Other:
- board size 20.5 x 20.8 mm -> 21.6 x 20.8 mm
- board text added: "+"
- board text added: "V8.0"
- board text added: "aux"
- board text added: "clk"
- board text added: "dio"
- board text added: "g"
- board text added: "gnd"
- board text added: "m10"
- board text added: "mathieu.p"
- board text added: "rst"
- board text added: "scl"
- board text added: "sda"
- board text added: "v"
