File: Hardware/hardware v8/hardware v8/hardware_V8.kicad_sch (KiCad schematic)
At the start: 36 parts, among them IC6 MLPF-WB-01E3, SW4 boot, U1 STM32WB55CGUx, Y1 830069528

Commit message: v8
Parts:
- removed C1, C3: 4.7u, Capacitor_SMD:C_0402_1005Metric, symbol Device:C_Small
- removed C12, C9: TBD, Capacitor_SMD:C_0201_0603Metric_Pad0.64x0.40mm_HandSolder, symbol Device:C_Small
- removed C17, C2, C21, C23: 100n, Capacitor_SMD:C_0201_0603Metric_Pad0.64x0.40mm_HandSolder, symbol Device:C_Small
- removed C22: 100p, Capacitor_SMD:C_0201_0603Metric_Pad0.64x0.40mm_HandSolder, symbol Device:C_Small
- removed IC6: MLPF-WB-01E3, samacsys2:BUMPLESS_CSP_2025, symbol samacsys2:MLPF-WB-01E3
- removed L1: 2.2u, Inductor_SMD:L_0805_2012Metric, symbol Device:L_Small
- removed L2: 10n, Inductor_SMD:L_0402_1005Metric, symbol Device:L_Small
- removed L3: L_Small, Inductor_SMD:L_0201_0603Metric_Pad0.64x0.40mm_HandSolder, symbol Device:L_Small
- removed L4: AMCA31-2R450G-S1F-T3, samacsys2:ANTC3216X140N, symbol samacsys2:AMCA31-2R450G-S1F-T3
- removed U1: STM32WB55CGUx, Package_DFN_QFN:QFN-48-1EP_7x7mm_P0.5mm_EP5.6x5.6mm, symbol MCU_ST_STM32WB:STM32WB55CGUx
- removed Y1: 830069528, samacsys:830069528, symbol samacsys:830069528
- added U1: STM32L432KCUx, Package_DFN_QFN:QFN-32-1EP_5x5mm_P0.5mm_EP3.45x3.45mm, symbol MCU_ST_STM32L4:STM32L432KCUx
Connections:
- net +3.3V: now also U1.1 (VDD), U1.17 (VDD), U1.5 (VDDA)
- net B1: now also U1.25 (PA15)
- net B2: now also U1.26 (PB3)
- net B_PW: now also U1.14 (PB0)
- net D+: now also U1.22 (PA12)
- net D-: now also U1.21 (PA11)
- net GND: now also U1.16 (VSS), U1.32 (VSS), U1.33 (VSS)
- net GPS_RX: now also U1.8 (PA2)
- net GPS_TX: now also U1.9 (PA3)
- net NRST: now also U1.4 (NRST)
- net OLED_SCL: now also U1.19 (PA9)
- net OLED_SDA: now also U1.20 (PA10)
- net SPI_CLK: now also U1.11 (PA5)
- net SPI_CS: now also U1.15 (PB1)
- net SPI_MISO: now also U1.12 (PA6)
- net SPI_MOSI: now also U1.13 (PA7)
- net SWCLK: now also U1.24 (PA14)
- net SWDIO: now also U1.23 (PA13)
- net at C8.1, R10.2, R16.2: now also U1.6 (PA0)
- net at R2.1: now also U1.29 (PB6)
- net at R1.1: now also U1.28 (PB5)
- net at C18.1, R6.1, SW4.1: now also U1.31 (PH3)
- new net AUX_EN: U1.10 (PA4)
- new net GPS_EN: U1.7 (PA1)
- new net USB_DETECT: U1.27 (PB4)
- no-connect marks 12 -> 0
Other:
- sheet BTN_CONN ports: added USB_DETECT; removed none
- sheet POWER ports: added AUX_EN, GPS_EN; removed none
- moved on the sheet: C10, C13, C15, C16, C18, C27, C8, LEDBLUE1, LEDGREEN1, R1, R10, R16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

Commit message: up
Connections:
- net B_PW: now also U1.6 (PA0); no longer U1.14 (PB0)
- net GPS_EXTINT: now reaches U1.18 (PA8)
- net ADC_BAT: now reaches C8.1, R10.2, R16.2
- net ADC_BAT: now also U1.14 (PB0); no longer U1.6 (PA0)
- no-connect marks 0 -> 4
Other:
- note added: "wakeup gpio PA0, PC13, PE6, PA2, PC5"
- moved on the sheet: C8, R10, R16
Changed lines of the file:
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@@
+		)
+	)
+	(text "wakeup gpio PA0, PC13, PE6, PA2, PC5"
+		(exclude_from_sim no)
+		(at 196.596 88.9 0)
+		(effects
+			(font
+				(size 1.27 1.27)
+			)
 		)
 	)
@@
 	)
 	(junction
-		(at 175.26 76.2)
+		(at 199.39 72.39)
 		(diameter 0)
 		(color 0 0 0 0)
@@
 	)
 	(junction
-		(at 175.26 81.28)
+		(at 199.39 77.47)
 		(diameter 0)
 		(color 0 0 0 0)
@@
 		(color 0 0 0 0)
 	)
-	(wire
-		(pts
-			(xy 175.26 73.66) (xy 175.26 76.2)
+	(no_connect
+		(at 332.74 40.64)
+	)
+	(no_connect
+		(at 125.73 109.22)
+	)
+	(no_connect
+		(at 125.73 88.9)
+	)
+	(no_connect
+		(at 125.73 86.36)
+	)
+	(wire
+		(pts
+			(xy 328.93 44.45) (xy 332.74 44.45)
+		)
+		(stroke
+			(width 0)
+			(type default)
+		)
+	)
+	(wire
+		(pts
+			(xy 199.39 69.85) (xy 199.39 72.39)
 		)
 		(stroke
@@
 	(wire
 		(pts
+			(xy 153.67 96.52) (xy 151.13 96.52)
+		)
+		(stroke
+			(width 0)
+			(type default)
+		)
+	)
+	(wire
+		(pts
 			(xy 121.92 68.58) (xy 124.46 68.58)
 		)
@@
 	(wire
 		(pts
-			(xy 184.15 76.2) (xy 175.26 76.2)
+			(xy 208.28 72.39) (xy 199.39 72.39)
 		)
 		(stroke
@@
 	(wire
 		(pts
-			(xy 184.15 81.28) (xy 175.26 81.28)
+			(xy 208.28 77.47) (xy 199.39 77.47)
 		)
 		(stroke
@@
 	(wire
 		(pts
+			(xy 153.67 76.2) (xy 151.13 76.2)
+		)
+		(stroke
+			(width 0)
+			(type default)
+		)
+	)
+	(wire
+		(pts
 			(xy 105.41 46.99) (xy 116.84 46.99)
 		)
@@
 	(wire
 		(pts
+			(xy 195.58 72.39) (xy 199.39 72.39)
+		)
+		(stroke
+			(width 0)
+			(type default)
+		)
+	)
+	(wire
+		(pts
 			(xy 116.84 46.99) (xy 130.81 46.99)
 		)
@@
 		(pts
 			(xy 115.57 116.84) (xy 110.49 116.84)
-		)
-		(stroke
-			(width 0)
-			(type default)
-		)
-	)
-	(wire
-		(pts
-			(xy 151.13 76.2) (xy 175.26 76.2)
 		)
 		(stroke
@@
 		)
 	)
+	(label "ADC_BAT"
+		(at 121.92 93.98 180)
+		(effects
+			(font
+				(size 1.27 1.27)
+			)
+			(justify right bottom)
+		)
+	)
 	(label "SPI_CLK"
 		(at 153.67 88.9 0)
@@
 		)
 	)
+	(label "GPS_EXTINT"
+		(at 328.93 44.45 180)
+		(effects
+			(font
+				(size 1.27 1.27)
+			)
+			(justify right bottom)
+		)
+	)
 	(label "GPS_EN"
 		(at 153.67 78.74 0)
@@
 		)
 	)
+	(label "B_PW"
+		(at 153.67 76.2 0)
+		(effects
+			(font
+				(size 1.27 1.27)
+			)
+			(justify left bottom)
+		)
+	)
 	(label "NRST"
 		(at 133.35 196.85 270)
@@
 		)
 	)
+	(label "GPS_EXTINT"
+		(at 153.67 96.52 0)
+		(effects
+			(font
+				(size 1.27 1.27)
+			)
+			(justify left bottom)
+		)
+	)
 	(label "GPS_RX"
 		(at 153.67 81.28 0)
@@
 		)
 	)
+	(label "ADC_BAT"
+		(at 195.58 72.39 180)
+		(effects
+			(font
+				(size 1.27 1.27)
+			)
+			(justify right bottom)
+		)
+	)
 	(label "SPI_CS"
 		(at 330.2 73.66 180)
@@
 	)
 	(label "B_PW"
-		(at 121.92 93.98 180)
-		(effects
-			(font
-				(size 1.27 1.27)
-			)
-			(justify right bottom)
-		)
-	)
-	(label "B_PW"
 		(at 328.93 161.29 180)
 		(effects
@@
 	(global_label "BAT+"
 		(shape input)
-		(at 175.26 68.58 90)
+		(at 199.39 64.77 90)
 		(fields_autoplaced yes)
 		(effects
@@
 		)
 		(property "Intersheetrefs" "${INTERSHEET_REFS}"
-			(at 175.26 60.6962 90)
+			(at 199.39 56.8862 90)
 			(effects
 				(font
@@
 	(symbol
 		(lib_id "power:GND")
-		(at 175.26 81.28 0)
+		(at 199.39 77.47 0)
 		(unit 1)
 		(exclude_from_sim no)
@@
 		(fields_autoplaced yes)
 		(property "Reference" "#PWR032"
-			(at 175.26 87.63 0)
+			(at 199.39 83.82 0)
 			(effects
 				(font
@@
 		)
 		(property "Value" "GND"
-			(at 175.26 86.36 0)
+			(at 199.39 82.55 0)
 			(effects
 				(font
@@
 		)
 		(property "Footprint" ""
-			(at 175.26 81.28 0)
+			(at 199.39 77.47 0)
 			(effects
 				(font
@@
 		)
 		(property "Datasheet" ""
-			(at 175.26 81.28 0)
+			(at 199.39 77.47 0)
 			(effects
 				(font
@@
 		)
 		(property "Description" "Power symbol creates a global label with name \"GND\" , ground"
-			(at 175.26 81.28 0)
+			(at 199.39 77.47 0)
 			(effects
 				(font
@@
 		(lib_name "R_Small_1")
 		(lib_id "Device:R_Small")
-		(at 184.15 78.74 180)
+		(at 208.28 74.93 180)
 		(unit 1)
 		(exclude_from_sim no)
@@
 		(fields_autoplaced yes)
 		(property "Reference" "R16"
-			(at 186.69 77.4699 0)
+			(at 210.82 73.6599 0)
 			(effects
 				(font
@@
 		)
 		(property "Value" "470k"
-			(at 186.69 80.0099 0)
+			(at 210.82 76.1999 0)
 			(effects
 				(font
@@
 		)
 		(property "Footprint" "Resistor_SMD:R_0201_0603Metric_Pad0.64x0.40mm_HandSolder"
-			(at 184.15 78.74 0)
+			(at 208.28 74.93 0)
 			(effects
 				(font
@@
 		)
 		(property "Datasheet" "~"
-			(at 184.15 78.74 0)
+			(at 208.28 74.93 0)
 			(effects
 				(font
@@
 		)
 		(property "Description" "Resistor, small symbol"
-			(at 184.15 78.74 0)
+			(at 208.28 74.93 0)
 			(effects
 				(font
@@
 		(lib_name "R_Small_1")
 		(lib_id "Device:R_Small")
-		(at 175.26 71.12 0)
+		(at 199.39 67.31 0)
 		(unit 1)
 		(exclude_from_sim no)
@@
 		(fields_autoplaced yes)
 		(property "Reference" "R10"
-			(at 177.8 69.8499 0)
+			(at 201.93 66.0399 0)
 			(effects
 				(font
@@
 		)
 		(property "Value" "470k"
-			(at 177.8 72.3899 0)
+			(at 201.93 68.5799 0)
 			(effects
 				(font
@@
 		)
 		(property "Footprint" "Resistor_SMD:R_0201_0603Metric_Pad0.64x0.40mm_HandSolder"
-			(at 175.26 71.12 0)
+			(at 199.39 67.31 0)
 			(effects
 				(font
@@
 		)
 		(property "Datasheet" "~"
-			(at 175.26 71.12 0)
+			(at 199.39 67.31 0)
 			(effects
 				(font
@@
 		)
 		(property "Description" "Resistor, small symbol"
-			(at 175.26 71.12 0)
+			(at 199.39 67.31 0)
 			(effects
 				(font
@@
 	(symbol
 		(lib_id "Device:C_Small")
-		(at 175.26 78.74 0)
+		(at 199.39 74.93 0)
 		(unit 1)
 		(exclude_from_sim no)
@@
 		(fields_autoplaced yes)
 		(property "Reference" "C8"
-			(at 177.8 77.4762 0)
+			(at 201.93 73.6662 0)
 			(effects
 				(font
@@
 		)
 		(property "Value" "100n"
-			(at 177.8 80.0162 0)
+			(at 201.93 76.2062 0)
 			(effects
 				(font
@@
 		)
 		(property "Footprint" "Capacitor_SMD:C_0201_0603Metric_Pad0.64x0.40mm_HandSolder"
-			(at 175.26 78.74 0)
+			(at 199.39 74.93 0)
 			(effects
 				(font
@@
 		)
 		(property "Datasheet" "~"
-			(at 175.26 78.74 0)
+			(at 199.39 74.93 0)
 			(effects
 				(font
@@
 		)
 		(property "Description" "Unpolarized capacitor, small symbol"
-			(at 175.26 78.74 0)
-			(effects
-				(font
+			(at 199.39 74.93 0)
+			(effects
+				(font

Commit message: up
Parts:
- R6: value 10k -> 20k
- TP3, TP4, TP5, TP6: now not fitted
Changed lines of the file:
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@@
 		(in_bom yes)
 		(on_board yes)
-		(dnp no)
+		(dnp yes)
 		(fields_autoplaced yes)
 		(property "Reference" "TP6"
@@
 		(in_bom yes)
 		(on_board yes)
-		(dnp no)
+		(dnp yes)
 		(fields_autoplaced yes)
 		(property "Reference" "TP5"
@@
 		(in_bom yes)
 		(on_board yes)
-		(dnp no)
+		(dnp yes)
 		(fields_autoplaced yes)
 		(property "Reference" "TP4"
@@
 			)
 		)
-		(property "Value" "10k"
+		(property "Value" "20k"
 			(at 88.9 87.6299 0)
 			(effects
@@
 		(in_bom yes)
 		(on_board yes)
-		(dnp no)
+		(dnp yes)
 		(fields_autoplaced yes)
 		(property "Reference" "TP3"

Commit message: up
Parts:
- LEDBLUE1, LEDGREEN1: Mouser Price/Stock (none) -> https://www.mouser.fr/ProductDetail/Wurth-Elektronik/150040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
- R1, R2: Mouser Part Number (none) -> 603-RC0201JR-07510RL; Mouser Price/Stock (none) -> https://www.mouser.fr/ProductDetail/YAGEO/RC0201JR-07510RL?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
- R10, R16: Mouser Part Number (none) -> 603-AC0201FR-07470KL; Mouser Price/Stock (none) -> https://www.mouser.fr/ProductDetail/YAGEO/AC0201FR-07470KL?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
- R6: Mouser Part Number (none) -> 603-AC0201FR-0720KL; Mouser Price/Stock (none) -> https://www.mouser.fr/ProductDetail/YAGEO/AC0201FR-0720KL?q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
- SW4: Mouser Part Number (none) -> 611-KXT341LHS; Mouser Price/Stock (none) -> https://www.mouser.fr/ProductDetail/CK/KXT-341-LHS?qs=W%2FM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
- U1: Mouser Part Number (none) -> 511-STM32L432KCU6; Mouser Price/Stock (none) -> https://www.mouser.fr/ProductDetail/STMicroelectronics/STM3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
Changed lines of the file:
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@@
+			)
+		)
+		(property "Mouser Part Number" "511-STM32L432KCU6"
+			(at 138.43 96.52 0)
+			(effects
+				(font
+					(size 1.27 1.27)
+				)
+				(hide yes)
+			)
+		)
+		(property "Mouser Price/Stock" "https://www.mouser.fr/ProductDetail/STMicroelectronics/STM32L432KCU6?qs=dTJS0cRn7oiybcTRwI97Tw%3D%3D"
+			(at 138.43 96.52 0)
+			(effects
+				(font
+					(size 1.27 1.27)
+				)
+				(hide yes)
 			)
 		)
@@
 		)
 		(property "Description" "Resistor, small symbol"
+			(at 208.28 74.93 0)
+			(effects
+				(font
+					(size 1.27 1.27)
+				)
+				(hide yes)
+			)
+		)
+		(property "Mouser Part Number" "603-AC0201FR-07470KL"
+			(at 208.28 74.93 0)
+			(effects
+				(font
+					(size 1.27 1.27)
+				)
+				(hide yes)
+			)
+		)
+		(property "Mouser Price/Stock" "https://www.mouser.fr/ProductDetail/YAGEO/AC0201FR-07470KL?qs=NgbZBzc1CyH0J6cte9SzFw%3D%3D"
 			(at 208.28 74.93 0)
 			(effects
@@
 			)
 		)
+		(property "Mouser Part Number" "603-RC0201JR-07510RL"
+			(at 107.95 116.84 90)
+			(effects
+				(font
+					(size 1.27 1.27)
+				)
+				(hide yes)
+			)
+		)
+		(property "Mouser Price/Stock" "https://www.mouser.fr/ProductDetail/YAGEO/RC0201JR-07510RL?qs=Q4gDqC5t5%2FDAdrMT21SmCw%3D%3D"
+			(at 107.95 116.84 90)
+			(effects
+				(font
+					(size 1.27 1.27)
+				)
+				(hide yes)
+			)
+		)
 		(pin "2"
 		)
@@
 		)
 		(property "Description" "Resistor, small symbol"
+			(at 199.39 67.31 0)
+			(effects
+				(font
+					(size 1.27 1.27)
+				)
+				(hide yes)
+			)
+		)
+		(property "Mouser Part Number" "603-AC0201FR-07470KL"
+			(at 199.39 67.31 0)
+			(effects
+				(font
+					(size 1.27 1.27)
+				)
+				(hide yes)
+			)
+		)
+		(property "Mouser Price/Stock" "https://www.mouser.fr/ProductDetail/YAGEO/AC0201FR-07470KL?qs=NgbZBzc1CyH0J6cte9SzFw%3D%3D"
 			(at 199.39 67.31 0)
 			(effects
@@
 			)
 		)
+		(property "Mouser Part Number" "603-RC0201JR-07510RL"
+			(at 107.95 107.95 90)
+			(effects
+				(font
+					(size 1.27 1.27)
+				)
+				(hide yes)
+			)
+		)
+		(property "Mouser Price/Stock" "https://www.mouser.fr/ProductDetail/YAGEO/RC0201JR-07510RL?qs=Q4gDqC5t5%2FDAdrMT21SmCw%3D%3D"
+			(at 107.95 107.95 90)
+			(effects
+				(font
+					(size 1.27 1.27)
+				)
+				(hide yes)
+			)
+		)
 		(pin "2"
 		)
@@
 			)
 		)
+		(property "Mouser Part Number" "603-AC0201FR-0720KL"
+			(at 86.36 86.36 0)
+			(effects
+				(font
+					(size 1.27 1.27)
+				)
+				(hide yes)
+			)
+		)
+		(property "Mouser Price/Stock" "https://www.mouser.fr/ProductDetail/YAGEO/AC0201FR-0720KL?qs=NgbZBzc1CyEbaKDOC3%252BFfg%3D%3D"
+			(at 86.36 86.36 0)
+			(effects
+				(font
+					(size 1.27 1.27)
+				)
+				(hide yes)
+			)
+		)
 		(pin "2"
 		)
@@
 			)
 		)
+		(property "Mouser Price/Stock" "https://www.mouser.fr/ProductDetail/Wurth-Elektronik/150040GS73240?qs=fAHHVMwC%252Bbgmx0FZHKuCJg%3D%3D"
+			(at 93.98 107.95 0)
+			(effects
+				(font
+					(size 1.27 1.27)
+				)
+				(hide yes)
+			)
+		)
 		(pin "2"
 		)
@@
 		(property "Description" "Push button switch, generic, two pins"
 			(at 86.36 76.2 0)
+			(effects
+				(font
+					(size 1.27 1.27)
+				)
+				(hide yes)
+			)
+		)
+		(property "Mouser Part Number" "611-KXT341LHS"
+			(at 86.36 76.2 90)
+			(effects
+				(font
+					(size 1.27 1.27)
+				)
+				(hide yes)
+			)
+		)
+		(property "Mouser Price/Stock" "https://www.mouser.fr/ProductDetail/CK/KXT-341-LHS?qs=W%2FMpXkg%252BdQ4NFpiYOsuiiw%3D%3D"
+			(at 86.36 76.2 90)
 			(effects
 				(font
@@
 			(at 93.98 116.84 0)
 			(effects
+				(font
+					(size 1.27 1.27)
+				)
+				(hide yes)
+			)
+		)
+		(property "Mouser Price/Stock" "https://www.mouser.fr/ProductDetail/Wurth-Elektronik/150040BS73240?qs=fAHHVMwC%252BbhvR%252BdBIVVrgw%3D%3D"
+			(at 93.98 116.84 0)
+			(effects
