File: Hardware/hardware v8/hardware v8/peripherial.kicad_sch (KiCad schematic)
At the start: 9 parts, among them IC2 W25Q128JVPIQ_TR, IC4 MAX-M10S-00B

Commit message: v8
Parts:
- removed IC2: W25Q128JVPIQ_TR, w25q128:SON127P600X500X80-9N-D, symbol winbond:W25Q128JVPIQ_TR
- added IC6: W25Q128JVPIQ, samacsys2:SON127P600X500X80-9N-D, symbol samacsys2:W25Q128JVPIQ
Connections:
- net GND: now also IC6.4 (GND_1), IC6.9 (GND_2)
- net SPI_CLK: now also IC6.6 (CLK)
- net SPI_CS: now also IC6.1 (~{CS})
- net SPI_MISO: now also IC6.2 (DO_(IO1))
- net SPI_MOSI: now also IC6.5 (DI_(IO0))
- net +3.3V renamed 3.3V_AUX
- net 3.3V_AUX: now also IC6.3 (~{WP_(IO2)}), IC6.7 (~{HOLD_OR_}/RESET_(IO3)), IC6.8 (VCC)
Other:
- moved on the sheet: C11, R13

Commit message: up
Connections:
- no-connect marks 8 -> 7
Changed lines of the file:
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@@
+	)
+	(junction
+		(at 105.41 208.28)
+		(diameter 0)
+		(color 0 0 0 0)
 	)
 	(junction
@@
 	)
 	(junction
-		(at 176.53 73.66)
-		(diameter 0)
-		(color 0 0 0 0)
-	)
-	(junction
 		(at 167.64 48.26)
 		(diameter 0)
@@
 	)
 	(no_connect
-		(at 184.15 73.66)
-	)
-	(no_connect
 		(at 152.4 71.12)
 	)
@@
 	(wire
 		(pts
-			(xy 96.52 208.28) (xy 107.95 208.28)
+			(xy 96.52 208.28) (xy 105.41 208.28)
 		)
 		(stroke
@@
 	(wire
 		(pts
-			(xy 184.15 73.66) (xy 176.53 73.66)
-		)
-		(stroke
-			(width 0)
-			(type default)
-		)
-	)
-	(wire
-		(pts
 			(xy 171.45 78.74) (xy 171.45 73.66)
 		)
@@
 		(pts
 			(xy 171.45 73.66) (xy 176.53 73.66)
+		)
+		(stroke
+			(width 0)
+			(type default)
+		)
+	)
+	(wire
+		(pts
+			(xy 105.41 208.28) (xy 107.95 208.28)
 		)
 		(stroke
@@
 					(unit 1)
 				)
+			)
+		)
+	)
+	(symbol
+		(lib_id "power:PWR_FLAG")
+		(at 105.41 208.28 180)
+		(unit 1)
+		(exclude_from_sim no)
+		(in_bom yes)
+		(on_board yes)
+		(dnp no)
+		(fields_autoplaced yes)
+		(property "Reference" "#FLG02"
+			(at 105.41 210.185 0)
+			(effects
+				(font
+					(size 1.27 1.27)
+				)
+				(hide yes)
+			)
+		)
+		(property "Value" "PWR_FLAG"
+			(at 105.41 213.36 0)
+			(effects
+				(font
+					(size 1.27 1.27)
+				)
+			)
+		)
+		(property "Footprint" ""
+			(at 105.41 208.28 0)
+			(effects
+				(font
+					(size 1.27 1.27)
+				)
+				(hide yes)
+			)
+		)
+		(property "Datasheet" "~"
+			(at 105.41 208.28 0)
+			(effects
+				(font
+					(size 1.27 1.27)
+				)
+				(hide yes)
+			)
+		)
+		(property "Description" "Special symbol for telling ERC where power comes from"
+			(at 105.41 208.28 0)
+			(effects
+				(font
+					(size 1.27 1.27)
+				)
+				(hide yes)
+			)
+		)
+		(pin "1"
+		)
+		(instances
+			(project ""
+				(path "/e491fdb3-646d-47e4-8ebb-9632fba4f524/84aae796-102b-48fc-8d1d-620f5c7b8bfd"
+					(reference "#FLG02")
+					(unit 1)
+				)

Commit message: up
Parts:
- added C2, C3: TBD, Capacitor_SMD:C_0402_1005Metric, symbol Device:C_Small
- added L1: TBD, Inductor_SMD:L_0402_1005Metric, symbol Device:L_Small
- added U3: 146235-0001, samacsys2:146235-0001, symbol samacsys2:146235-0001
Connections:
- net GND: now also C2.2, C3.2
- net at IC4.11 (RF_IN): now also C2.1, L1.2
- new net: C3.1, L1.1, U3.1
- no-connect marks 7 -> 10

Commit message: up
Parts:
- C2: value TBD -> 1.8nH
- C3: now not fitted
- L1: value TBD -> 5.1nH
- R13: value 10k -> 20k
Changed lines of the file:
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@@
 		(in_bom yes)
 		(on_board yes)
-		(dnp no)
+		(dnp yes)
 		(fields_autoplaced yes)
 		(property "Reference" "C3"
@@
 			)
 		)
-		(property "Value" "TBD"
+		(property "Value" "5.1nH"
 			(at 86.36 73.66 90)
 			(effects
@@
 			)
 		)
-		(property "Value" "TBD"
+		(property "Value" "1.8nH"
 			(at 93.98 80.0162 0)
 			(effects
@@
 		(fields_autoplaced yes)
 		(property "Reference" "R13"
-			(at 158.75 213.3601 0)
+			(at 163.83 210.8199 0)
 			(effects
 				(font
 					(size 1.016 1.016)
 				)
-				(justify right)
-			)
-		)
-		(property "Value" "10k"
-			(at 158.75 210.8201 0)
-			(effects
-				(font
-					(size 1.27 1.27)
-				)
-				(justify right)
-			)
-		)
+				(justify left)
+			)
+		)
+		(property "Value" "20k"
+			(at 163.83 213.3599 0)
+			(effects
+				(font
+					(size 1.27 1.27)
+				)
+				(justify left)
+			)
+		)

Commit message: up
Parts:
- R11, R12: Mouser Part Number (none) -> 603-RC0201JR-07510RL; Mouser Price/Stock (none) -> https://www.mouser.fr/ProductDetail/YAGEO/RC0201JR-07510RL?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
- R13: Mouser Part Number (none) -> 603-AC0201FR-0720KL; Mouser Price/Stock (none) -> https://www.mouser.fr/ProductDetail/YAGEO/AC0201FR-0720KL?q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
Changed lines of the file:
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@@
+			)
+		)
+		(property "Mouser Part Number" "603-RC0201JR-07510RL"
+			(at 161.29 86.36 90)
+			(effects
+				(font
+					(size 1.27 1.27)
+				)
+				(hide yes)
+			)
+		)
+		(property "Mouser Price/Stock" "https://www.mouser.fr/ProductDetail/YAGEO/RC0201JR-07510RL?qs=Q4gDqC5t5%2FDAdrMT21SmCw%3D%3D"
+			(at 161.29 86.36 90)
+			(effects
+				(font
+					(size 1.27 1.27)
+				)
+				(hide yes)
 			)
 		)
@@
 		(property "Description" "Resistor, small symbol"
 			(at 166.37 90.17 0)
+			(effects
+				(font
+					(size 1.27 1.27)
+				)
+				(hide yes)
+			)
+		)
+		(property "Mouser Part Number" "603-RC0201JR-07510RL"
+			(at 166.37 90.17 90)
+			(effects
+				(font
+					(size 1.27 1.27)
+				)
+				(hide yes)
+			)
+		)
+		(property "Mouser Price/Stock" "https://www.mouser.fr/ProductDetail/YAGEO/RC0201JR-07510RL?qs=Q4gDqC5t5%2FDAdrMT21SmCw%3D%3D"
+			(at 166.37 90.17 90)
 			(effects
 				(font
@@
 			(at 161.29 212.09 0)
 			(effects
+				(font
+					(size 1.27 1.27)
+				)
+				(hide yes)
+			)
+		)
+		(property "Mouser Part Number" "603-AC0201FR-0720KL"
+			(at 161.29 212.09 0)
+			(effects
+				(font
+					(size 1.27 1.27)
+				)
+				(hide yes)
+			)
+		)
+		(property "Mouser Price/Stock" "https://www.mouser.fr/ProductDetail/YAGEO/AC0201FR-0720KL?qs=NgbZBzc1CyEbaKDOC3%252BFfg%3D%3D"
+			(at 161.29 212.09 0)
+			(effects
