File: Hardware/hardware v8/hardware v8/untitled.kicad_sch (KiCad schematic)
At the start: 10 parts, among them IC3 LDO40LPU33RY, IC5 LTC4065EDC#TRMPBF

Commit message: v8
Parts:
- removed D1: ~, LED_SMD:LED_0201_0603Metric_Pad0.64x0.40mm_HandSolder, symbol Device:LED_Small
- removed IC3: LDO40LPU33RY, samacsys:SON95P300X300X90-7N-D, symbol ldo40pury:LDO40LPU33RY
- added C1: 1u, Capacitor_SMD:C_0402_1005Metric, symbol Device:C
- added IC1: TPS22960RSER, samacsys2:TPS22960RSER, symbol samacsys2:TPS22960RSER
- added LEDRED1: 150040RS73240, LED_SMD:LED_0402_1005Metric, symbol Device:LED_Small
- added R20, R21: 10k, Resistor_SMD:R_0201_0603Metric_Pad0.64x0.40mm_HandSolder, symbol Device:R_Small
- added U2: ldln025pu, samacsys:ldln025pu, symbol samacsys:ldln025pu
Connections:
- net +3.3V: now also C1.1, IC1.1 (VIN1), IC1.3 (SR), IC1.8 (VIN2), U2.1 (VOUT)
- net BAT+: now also U2.4 (VIN); no longer R5.1
- net GND: now also R5.1, C1.2, IC1.6 (GND), R20.1, R21.1, U2.2 (GND)
- net at R4.1: now also LEDRED1.2 (A)
- net at R18.1, R5.2: now also U2.3 (EN)
- net at IC5.2 (~{CHRG}): now also LEDRED1.1 (K)
- new net 3.3V_AUX: IC1.4 (VOUT1)
- new net 3.3V_GPS: IC1.5 (VOUT2)
- new net AUX_EN: IC1.2 (ON1), R21.2
- new net GPS_EN: IC1.7 (ON2), R20.2
Other:
- note added: "660us rise time"

Commit message: up
Parts:
- R20, R21: value 10k -> 100k
Connections:
- no-connect marks 1 -> 0
Changed lines of the file:
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@@
+	)
+	(junction
+		(at 184.15 64.77)
+		(diameter 0)
+		(color 0 0 0 0)
 	)
 	(junction
@@
 	)
 	(junction
+		(at 219.71 105.41)
+		(diameter 0)
+		(color 0 0 0 0)
+	)
+	(junction
 		(at 58.42 45.72)
 		(diameter 0)
@@
 		(color 0 0 0 0)
 	)
-	(no_connect
-		(at 105.41 46.99)
-	)
 	(wire
 		(pts
@@
 	(wire
 		(pts
-			(xy 175.26 64.77) (xy 198.12 64.77)
+			(xy 175.26 64.77) (xy 184.15 64.77)
 		)
 		(stroke
@@
 	(wire
 		(pts
+			(xy 184.15 64.77) (xy 198.12 64.77)
+		)
+		(stroke
+			(width 0)
+			(type default)
+		)
+	)
+	(wire
+		(pts
 			(xy 198.12 64.77) (xy 198.12 80.01)
 		)
@@
 	(wire
 		(pts
+			(xy 219.71 107.95) (xy 219.71 105.41)
+		)
+		(stroke
+			(width 0)
+			(type default)
+		)
+	)
+	(wire
+		(pts
 			(xy 209.55 64.77) (xy 219.71 64.77)
 		)
@@
 		(pts
 			(xy 116.84 45.72) (xy 125.73 45.72)
+		)
+		(stroke
+			(width 0)
+			(type default)
+		)
+	)
+	(wire
+		(pts
+			(xy 219.71 105.41) (xy 219.71 102.87)
 		)
 		(stroke
@@
 	(global_label "3.3V_AUX"
 		(shape input)
-		(at 219.71 102.87 0)
+		(at 219.71 107.95 0)
 		(fields_autoplaced yes)
 		(effects
@@
 		)
 		(property "Intersheetrefs" "${INTERSHEET_REFS}"
-			(at 231.4038 102.87 0)
+			(at 231.4038 107.95 0)
 			(effects
 				(font
@@
 			)
 			(justify left)
+		)
+	)
+	(symbol
+		(lib_id "power:PWR_FLAG")
+		(at 219.71 105.41 90)
+		(unit 1)
+		(exclude_from_sim no)
+		(in_bom yes)
+		(on_board yes)
+		(dnp no)
+		(fields_autoplaced yes)
+		(property "Reference" "#FLG03"
+			(at 217.805 105.41 0)
+			(effects
+				(font
+					(size 1.27 1.27)
+				)
+				(hide yes)
+			)
+		)
+		(property "Value" "PWR_FLAG"
+			(at 215.9 105.4099 90)
+			(effects
+				(font
+					(size 1.27 1.27)
+				)
+				(justify left)
+			)
+		)
+		(property "Footprint" ""
+			(at 219.71 105.41 0)
+			(effects
+				(font
+					(size 1.27 1.27)
+				)
+				(hide yes)
+			)
+		)
+		(property "Datasheet" "~"
+			(at 219.71 105.41 0)
+			(effects
+				(font
+					(size 1.27 1.27)
+				)
+				(hide yes)
+			)
+		)
+		(property "Description" "Special symbol for telling ERC where power comes from"
+			(at 219.71 105.41 0)
+			(effects
+				(font
+					(size 1.27 1.27)
+				)
+				(hide yes)
+			)
+		)
+		(pin "1"
+		)
+		(instances
+			(project "hardware_V8"
+				(path "/e491fdb3-646d-47e4-8ebb-9632fba4f524/42e3e1b1-9911-4d5d-8c18-366c2d58b563"
+					(reference "#FLG03")
+					(unit 1)
+				)
+			)
 		)
 	)
@@
 			)
 		)
-		(property "Value" "10k"
+		(property "Value" "100k"
 			(at 185.42 90.1699 0)
 			(effects
@@
 	)
 	(symbol
+		(lib_id "power:PWR_FLAG")
+		(at 184.15 64.77 0)
+		(unit 1)
+		(exclude_from_sim no)
+		(in_bom yes)
+		(on_board yes)
+		(dnp no)
+		(fields_autoplaced yes)
+		(property "Reference" "#FLG05"
+			(at 184.15 62.865 0)
+			(effects
+				(font
+					(size 1.27 1.27)
+				)
+				(hide yes)
+			)
+		)
+		(property "Value" "PWR_FLAG"
+			(at 184.15 59.69 0)
+			(effects
+				(font
+					(size 1.27 1.27)
+				)
+			)
+		)
+		(property "Footprint" ""
+			(at 184.15 64.77 0)
+			(effects
+				(font
+					(size 1.27 1.27)
+				)
+				(hide yes)
+			)
+		)
+		(property "Datasheet" "~"
+			(at 184.15 64.77 0)
+			(effects
+				(font
+					(size 1.27 1.27)
+				)
+				(hide yes)
+			)
+		)
+		(property "Description" "Special symbol for telling ERC where power comes from"
+			(at 184.15 64.77 0)
+			(effects
+				(font
+					(size 1.27 1.27)
+				)
+				(hide yes)
+			)
+		)
+		(pin "1"
+		)
+		(instances
+			(project "hardware_V8"
+				(path "/e491fdb3-646d-47e4-8ebb-9632fba4f524/42e3e1b1-9911-4d5d-8c18-366c2d58b563"
+					(reference "#FLG05")
+					(unit 1)
+				)
+			)
+		)
+	)
+	(symbol
 		(lib_name "R_Small_1")
 		(lib_id "Device:R_Small")
@@
 			)
 		)
-		(property "Value" "10k"
+		(property "Value" "100k"
 			(at 250.19 83.8199 0)
 			(effects

Commit message: up
Parts:
- R18: value 10k -> 120k
- R5: value 10k -> 20k
Other:
- note added: "VIH MIN 1.2V VIL MAX 0.4V"
- note added: "a tester (cutoff a 2.8V) si probleme R18 prend 0R"
Changed lines of the file:
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@@
+		)
+	)
+	(text "VIH MIN 1.2V\nVIL MAX 0.4V"
+		(exclude_from_sim no)
+		(at 66.294 71.374 0)
+		(effects
+			(font
+				(size 1.27 1.27)
+			)
 		)
 	)
@@
 		(exclude_from_sim no)
 		(at 65.786 33.528 0)
+		(effects
+			(font
+				(size 1.27 1.27)
+			)
+		)
+	)
+	(text "a tester (cutoff a 2.8V) si probleme R18 prend 0R"
+		(exclude_from_sim no)
+		(at 60.452 77.724 0)
 		(effects
 			(font
@@
 			)
 		)
-		(property "Value" "10k"
+		(property "Value" "20k"
 			(at 68.58 58.4199 0)
 			(effects
@@
 			)
 		)
-		(property "Value" "10k"
+		(property "Value" "120k"
 			(at 68.58 50.7999 0)
 			(effects

Commit message: up
Parts:
- LEDRED1: Mouser Price/Stock (none) -> https://www.mouser.fr/ProductDetail/Wurth-Elektronik/150040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
- R17, R5: Mouser Part Number (none) -> 603-AC0201FR-0720KL; Mouser Price/Stock (none) -> https://www.mouser.fr/ProductDetail/YAGEO/AC0201FR-0720KL?q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
- R18: Mouser Part Number (none) -> 603-RC0201JR-07120KL; Mouser Price/Stock (none) -> https://www.mouser.fr/ProductDetail/YAGEO/RC0201JR-07120KL?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
- R20, R21: Mouser Part Number (none) -> 603-RC0201BR-07100KL; Mouser Price/Stock (none) -> https://www.mouser.fr/ProductDetail/YAGEO/RC0201BR-07100KL?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
- R4: Mouser Part Number (none) -> 603-RC0201JR-07510RL; Mouser Price/Stock (none) -> https://www.mouser.fr/ProductDetail/YAGEO/RC0201JR-07510RL?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
- U2: Mouser Part Number (none) -> 511-LDLN025PU33R; Mouser Price/Stock (none) -> https://www.mouser.fr/ProductDetail/STMicroelectronics/LDLN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
Changed lines of the file:
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@@
+			)
+		)
+		(property "Mouser Part Number" "603-RC0201JR-07510RL"
+			(at 38.1 143.51 0)
+			(effects
+				(font
+					(size 1.27 1.27)
+				)
+				(hide yes)
+			)
+		)
+		(property "Mouser Price/Stock" "https://www.mouser.fr/ProductDetail/YAGEO/RC0201JR-07510RL?qs=Q4gDqC5t5%2FDAdrMT21SmCw%3D%3D"
+			(at 38.1 143.51 0)
+			(effects
+				(font
+					(size 1.27 1.27)
+				)
+				(hide yes)
 			)
 		)
@@
 			)
 		)
+		(property "Mouser Part Number" "603-AC0201FR-0720KL"
+			(at 66.04 57.15 0)
+			(effects
+				(font
+					(size 1.27 1.27)
+				)
+				(hide yes)
+			)
+		)
+		(property "Mouser Price/Stock" "https://www.mouser.fr/ProductDetail/YAGEO/AC0201FR-0720KL?qs=NgbZBzc1CyEbaKDOC3%252BFfg%3D%3D"
+			(at 66.04 57.15 0)
+			(effects
+				(font
+					(size 1.27 1.27)
+				)
+				(hide yes)
+			)
+		)
 		(pin "2"
 		)
@@
 			)
 		)
+		(property "Mouser Part Number" "603-RC0201BR-07100KL"
+			(at 182.88 88.9 0)
+			(effects
+				(font
+					(size 1.27 1.27)
+				)
+				(hide yes)
+			)
+		)
+		(property "Mouser Price/Stock" "https://www.mouser.fr/ProductDetail/YAGEO/RC0201BR-07100KL?qs=r5DSvlrkXmKB5tn%2FBtA0vQ%3D%3D"
+			(at 182.88 88.9 0)
+			(effects
+				(font
+					(size 1.27 1.27)
+				)
+				(hide yes)
+			)
+		)
 		(pin "2"
 		)
@@
 		)
 		(property "Description" ""
+			(at 90.17 52.07 0)
+			(effects
+				(font
+					(size 1.27 1.27)
+				)
+				(hide yes)
+			)
+		)
+		(property "Mouser Part Number" "511-LDLN025PU33R"
+			(at 90.17 52.07 0)
+			(effects
+				(font
+					(size 1.27 1.27)
+				)
+				(hide yes)
+			)
+		)
+		(property "Mouser Price/Stock" "https://www.mouser.fr/ProductDetail/STMicroelectronics/LDLN025PU33R?qs=aVyJF2WnouRLo66BkrxZ7g%3D%3D"
 			(at 90.17 52.07 0)
 			(effects
@@
 			)
 		)
+		(property "Mouser Price/Stock" "https://www.mouser.fr/ProductDetail/Wurth-Elektronik/150040GS73240?qs=fAHHVMwC%252Bbgmx0FZHKuCJg%3D%3D"
+			(at 49.53 143.51 0)
+			(effects
+				(font
+					(size 1.27 1.27)
+				)
+				(hide yes)
+			)
+		)
 		(pin "2"
 		)
@@
 		)
 		(property "Description" "Resistor, small symbol"
+			(at 247.65 82.55 0)
+			(effects
+				(font
+					(size 1.27 1.27)
+				)
+				(hide yes)
+			)
+		)
+		(property "Mouser Part Number" "603-RC0201BR-07100KL"
+			(at 247.65 82.55 0)
+			(effects
+				(font
+					(size 1.27 1.27)
+				)
+				(hide yes)
+			)
+		)
+		(property "Mouser Price/Stock" "https://www.mouser.fr/ProductDetail/YAGEO/RC0201BR-07100KL?qs=r5DSvlrkXmKB5tn%2FBtA0vQ%3D%3D"
 			(at 247.65 82.55 0)
 			(effects
@@
 			)
 		)
+		(property "Mouser Part Number" "603-AC0201FR-0720KL"
+			(at 92.71 140.97 90)
+			(effects
+				(font
+					(size 1.27 1.27)
+				)
+				(hide yes)
+			)
+		)
+		(property "Mouser Price/Stock" "https://www.mouser.fr/ProductDetail/YAGEO/AC0201FR-0720KL?qs=NgbZBzc1CyEbaKDOC3%252BFfg%3D%3D"
+			(at 92.71 140.97 90)
+			(effects
+				(font
+					(size 1.27 1.27)
+				)
+				(hide yes)
+			)
+		)
 		(pin "2"
 		)
@@
 			(at 66.04 49.53 0)
 			(effects
+				(font
+					(size 1.27 1.27)
+				)
+				(hide yes)
+			)
+		)
+		(property "Mouser Part Number" "603-RC0201JR-07120KL"
+			(at 66.04 49.53 0)
+			(effects
+				(font
+					(size 1.27 1.27)
+				)
+				(hide yes)
+			)
+		)
+		(property "Mouser Price/Stock" "https://www.mouser.fr/ProductDetail/YAGEO/RC0201JR-07120KL?qs=50q%252BZR8McTE42SrRwjbjMg%3D%3D"
+			(at 66.04 49.53 0)
+			(effects
