File: Hardware/hardware_v9/hardware v8/hardware_V8.kicad_sch (KiCad schematic)
At the start: 19 parts, among them SW4 boot, U1 STM32L432KCUx

Commit message: up
Parts:
- removed C18: 100n, Capacitor_SMD:C_0201_0603Metric_Pad0.64x0.40mm_HandSolder, symbol Device:C_Small
- removed R6: 20k, Resistor_SMD:R_0201_0603Metric_Pad0.64x0.40mm_HandSolder, symbol Device:R_Small
- removed SW4: boot, samacsys:KXT341LHS, symbol Switch:SW_Push
- C16: footprint Capacitor_SMD:C_0402_1005Metric -> Capacitor_SMD:C_0201_0603Metric_Pad0.64x0.40mm_HandSolder
Connections:
- net GPS_EXTINT is gone; now on net USB_DETECT: U1.18 (PA8)
- net ADC_BAT: now also U1.7 (PA1); no longer U1.14 (PB0)
- net AUX_EN: now also U1.15 (PB1); no longer U1.10 (PA4)
- net B1: now also U1.31 (PH3); no longer U1.25 (PA15)
- net GPS_EN: now also U1.14 (PB0); no longer U1.7 (PA1)
- net SPI_CS: now also U1.10 (PA4); no longer U1.15 (PB1)
- net USB_DETECT: no longer U1.27 (PB4)
- new net SD_DET: U1.27 (PB4)
- no-connect marks 3 -> 4
Other:
- sheet Peripherial ports: added SD_Detect; removed GPS_EXT
