File: Hardware/hardware_v9/hardware v8/peripherial.kicad_sch (KiCad schematic)
At the start: 11 parts, among them IC4 MAX-M10S-00B, IC6 W25Q128JVPIQ

Commit message: up
Parts:
- removed C25, C26: 100n, Capacitor_SMD:C_0201_0603Metric_Pad0.64x0.40mm_HandSolder, symbol Device:C_Small
- removed C28: 4.7u, Capacitor_SMD:C_0402_1005Metric, symbol Device:C_Small
- removed IC4: MAX-M10S-00B, samacsys:MAXM10S00B, symbol samacsys:MAX-M10S-00B
- removed IC6: W25Q128JVPIQ, samacsys2:SON127P600X500X80-9N-D, symbol samacsys2:W25Q128JVPIQ
- removed R11, R12: 510R, Resistor_SMD:R_0201_0603Metric_Pad0.64x0.40mm_HandSolder, symbol Device:R_Small
- removed R8: 0R, Resistor_SMD:R_0402_1005Metric, symbol Device:R_Small
- removed U3: ~, samacsys2:GNSS_8mmx8mm, symbol samacsys2:GNSS_antenna_8mmx8mm
- added C12: 1u, Capacitor_SMD:C_0201_0603Metric_Pad0.64x0.40mm_HandSolder, symbol Device:C_Small
- added C21: 4.7u, Capacitor_SMD:C_0402_1005Metric, symbol Device:C_Small
- added J1: Micro_SD_Card_Det2, Connector_Card:microSD_HC_Molex_104031-0811, symbol Connector:Micro_SD_Card_Det2
- added PA1010D1: PA1010D, pa1010d:PA1010D, symbol PA1010D:PA1010D
- added R14, R15: 470R, Resistor_SMD:R_0201_0603Metric_Pad0.64x0.40mm_HandSolder, symbol Device:R_Small
- added R24: 0R, Resistor_SMD:R_0201_0603Metric_Pad0.64x0.40mm_HandSolder, symbol Device:R_Small
- added R25: 20k, Resistor_SMD:R_0201_0603Metric_Pad0.64x0.40mm_HandSolder, symbol Device:R_Small
- added R26: 22R, Resistor_SMD:R_0201_0603Metric_Pad0.64x0.40mm_HandSolder, symbol Device:R_Small
Connections:
- net 3.3V_AUX: now also C21.1, J1.4 (VDD), R25.2; no longer C11.1
- net 3.3V_GPS: now also C12.1, PA1010D1.10 (VCC)
- net BAT+: now also R24.1
- net GND: now also C12.2, C21.2, J1.10 (DET_A), J1.6 (VSS), J1.SH (SHIELD), PA1010D1.7 (GND)
- net GPS_RX: now also R14.2
- net GPS_TX: now also R15.1
- net SPI_CLK: now also R26.1
- net SPI_CS: now also J1.2 (DAT3/CD)
- net SPI_MISO: now also J1.7 (DAT0)
- net SPI_MOSI: now also J1.3 (CMD)
- new net: J1.5 (CLK), R26.2
- new net: PA1010D1.4 (TX), R15.2
- new net: PA1010D1.5 (RX), R14.1
- new net: PA1010D1.9 (VBACKUP), R24.2
- new net SD_Detect: C11.1, J1.9 (DET_B), R25.1
- no-connect marks 8 -> 7
Other:
- note added: "PILE lithium de backup"
- note removed: "MEMOIRE SPI"
