File: Hardware/hardware_v9/hardware v8/untitled.kicad_sch (KiCad schematic)
At the start: 13 parts, among them IC1 TPS22960RSER, IC5 LTC4065EDC#TRMPBF, U2 ldln025pu

Commit message: up
Parts:
- C1, C29, C4: footprint Capacitor_SMD:C_0402_1005Metric -> Capacitor_SMD:C_0201_0603Metric_Pad0.64x0.40mm_HandSolder

Commit message: up
Parts:
- removed IC1: TPS22960RSER, samacsys2:TPS22960RSER, symbol samacsys2:TPS22960RSER
- removed R20: 100k, Resistor_SMD:R_0201_0603Metric_Pad0.64x0.40mm_HandSolder, symbol Device:R_Small
- added C2, C3, C5, C6: 1u, Capacitor_SMD:C_0201_0603Metric_Pad0.64x0.40mm_HandSolder, symbol Device:C
- added R27: 100k, Resistor_SMD:R_0201_0603Metric_Pad0.64x0.40mm_HandSolder, symbol Device:R_Small
- added U3, U5: ldln025pu, samacsys:ldln025pu, symbol samacsys:ldln025pu
Connections:
- net +3.3V: now also C2.1; no longer C1.1
- net 3.3V_AUX: now also C1.1, U5.1 (VOUT)
- net 3.3V_GPS: now also C5.1, U3.1 (VOUT)
- net AUX_EN: now also U5.3 (EN)
- net BAT+: now also C3.1, C6.1, U3.4 (VIN), U5.4 (VIN)
- net GND: now also C2.2, C3.2, C5.2, C6.2, R27.1, U3.2 (GND), U5.2 (GND)
- net GPS_EN: now also R27.2, U3.3 (EN)
Other:
- note removed: "660us rise time"
