File: Hardware/hardware_v9/hardware v9/hardware_V9.kicad_sch (KiCad schematic)
At the start: 17 parts, among them U1 STM32L432KCUx

Commit message: up
Other:
- note added: "STM32L432"
- note removed: "STM32WB55"
Changed lines of the file:
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@@
 		)
 	)
-	(text "STM32WB55"
+	(text "STM32L432"
 		(exclude_from_sim no)
 		(at 22.86 20.32 0)
