File: Hardware/aux_flex_pcb/aux_flex_pcb.kicad_pcb (KiCad board)
At the start: 6 copper layers, 0 parts

Commit message: up
Routing:
- net /B_PW: track 19.7 -> 0.00 mm
- net /B1: track 18.8 -> 0.00 mm
- net /SD_DET: track 16.9 -> 0.00 mm
- net +3.3V: track 14.5 -> 0.00 mm
- net /SPI_CS: track 13.6 -> 0.00 mm
- net 3.3V_AUX: track 13.3 -> 0.00 mm
- net Net-(PA1010D1-VBACKUP): track 12.8 -> 0.00 mm
- net Net-(LEDGREEN1-A): track 8.63 -> 0.00 mm
- net Net-(PA1010D1-TX): track 8.33 -> 0.00 mm
- net Net-(PA1010D1-RX): track 7.58 -> 0.00 mm
- net Net-(LEDBLUE1-A): track 6.68 -> 0.00 mm
- net /OLED_SCL: track 3.20 -> 0.00 mm
- net /OLED_SDA: track 3.00 -> 0.00 mm
- removed copper zone on In3.Cu, net +3.3V
- removed copper zone on In3.Cu, net 3.3V_AUX
- removed copper zone on In3.Cu, net BAT+
- removed copper zone on In3.Cu, net GND
- removed copper zone on In3.Cu, net vusb
Other:
- copper layers 6 -> 2

Commit message: up
Parts:
- added C14: 100n, Capacitor_SMD:C_0201_0603Metric_Pad0.64x0.40mm_HandSolder, F.Cu at (144.9, 101.7)
- added J1: 503552-0622, samacsys2:5035520622, B.Cu at (140.1, 108.3)
- added J2: 503548-0622, samacsys2:5035480622, F.Cu at (140.1, 108.3)
- added R19: 470k, Resistor_SMD:R_0201_0603Metric_Pad0.64x0.40mm_HandSolder, F.Cu at (144.9, 105.2)
- added R3: 470k, Resistor_SMD:R_0201_0603Metric_Pad0.64x0.40mm_HandSolder, F.Cu at (144.9, 103.4)
- added TP1: TestPoint, samacsys2:1mm_circle, F.Cu at (143.7, 107.4)
- added TP2: TestPoint, samacsys2:1mm_circle, F.Cu at (143.7, 109.4)
