File: Hardware/aux_flex_pcb/aux_flex_pcb.kicad_pcb (KiCad board)
At the start: 2 copper layers, 22 parts, among them IC2 XB5353A, J2 BM29B-2DP_2-0.35V_53_, J3 BM29B-2DP_2-0.35V_53_, J4 503552-0622, U1 ldln025pu, U2 DA14531-00000FX2, Y1 830108254201

Commit message: up
Parts:
- removed ANT1: 2450AT14A0100001T, samacsys2:2450AT14A0100001T
- J2, J3, J4, TP5, TP6, TP7, TP8: moved to B.Cu
- moved C21 32.2 mm to (169.8, 105.1)
- moved C23 30.3 mm to (166.4, 109.8), turned to 90 degrees
- moved L2 29.7 mm to (165.2, 109.1), turned to -90 degrees
- moved C25 29.6 mm to (169.8, 106.0)
- moved C22 29.6 mm to (165.6, 107.8)
- moved J3 29.5 mm to (173.9, 117.5), turned to 180 degrees
- moved J2 29.4 mm to (170.6, 117.5), turned to 180 degrees
- moved C27 28.0 mm to (168.2, 102.4), turned to 90 degrees
- moved C26 28.0 mm to (169.8, 104.3)
- moved C19 27.8 mm to (161.1, 105.9)
- moved R22 25.9 mm to (169.9, 101.4), turned to 180 degrees
- moved Y1 25.7 mm to (167.8, 107.6)
- moved TP5 25.5 mm to (170.4, 104.3), turned to 180 degrees
- moved TP6 23.2 mm to (168.5, 105.0), turned to 180 degrees
- moved R21 22.7 mm to (161.1, 105.2), turned to 180 degrees
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Connections:
- C23 pad 1: Net-(ANT1-FEED) -> unconnected-(C23-Pad1)
- L2 pad 2: Net-(ANT1-FEED) -> unconnected-(C23-Pad1)
- Y1 pad 1: Net-(U2B-XTAL32Mm) -> Net-(U2B-XTAL32Mp)
- Y1 pad 3: Net-(U2B-XTAL32Mp) -> Net-(U2B-XTAL32Mm)
Routing:
- net unconnected-(C23-Pad1): track 0.00 -> 25.6 mm
- net /exti: track 0.00 -> 10.0 mm, vias 0 -> 1
- net /rx_sup: track 0.00 -> 5.95 mm, vias 0 -> 2
- net /tx_sup: track 0.00 -> 2.68 mm, vias 0 -> 1
- net Net-(U2B-XTAL32Mm): track 0.00 -> 2.40 mm
- net /RF: track 0.00 -> 2.31 mm
- net Net-(U2B-XTAL32Mp): track 0.00 -> 2.31 mm
- net 3.3V_AUX: track 0.00 -> 2.15 mm, vias 0 -> 1
- net /SWCLK: track 0.00 -> 1.95 mm, vias 0 -> 1
- net /SWDIO: track 0.00 -> 1.01 mm, vias 0 -> 1
- net GND: vias 0 -> 15
- added copper zone on F.Cu, net 3.3V_AUX
- added copper zone on B.Cu, net GND
- added copper zone on F.Cu, net GND
- added copper zone on F.Cu, net Net-(U1-VOUT)
Other:
- board outline added: 15.4 x 17.7 mm

Commit message: up
Parts:
- removed TP5: gnd, samacsys2:1mm_circle
- TP6, TP7, TP8: moved to F.Cu
- moved TP7 5.15 mm to (169.8, 107.1), turned to 0 degrees
- moved R21 4.23 mm to (161.6, 109.4), turned to 90 degrees
- moved C19 2.16 mm to (161.6, 103.8)
- moved IC2 2.00 mm to (161.6, 106.4)
- moved J2 0.40 mm to (170.6, 117.9)
- moved J3 0.40 mm to (173.9, 117.9)
- moved TP6 0.17 mm to (168.3, 105.0), turned to 0 degrees
- turned TP8 to 0 degrees
Connections:
- J2 pad 3: /ADC_SUP -> unconnected-(J2-Pad3)
- J2 pad 4: /ADC_SUP -> unconnected-(J2-Pad4)
- J3 pad 5: BAT+ -> BAT1+
- J3 pad 6: BAT+ -> BAT1+
- J4 pad 3: /exti -> /P-
- R22 pad 2: /exti -> /P-
- U1 pad 3: /exti -> /P-
Routing:
- net GND: track 0.00 -> 25.8 mm, vias 15 -> 18
- net BAT+: track 0.00 -> 17.6 mm, vias 0 -> 2
- net /P-: track 0.00 -> 11.9 mm, vias 0 -> 8
- net /exti: track 10.0 -> 0.00 mm, vias 1 -> 0
- net /SWCLK: track 1.95 -> 7.92 mm, vias 1 -> 2
- net Net-(IC2-VDD): track 0.00 -> 5.81 mm
- net BAT1+: vias 0 -> 1
- added copper zone on B.Cu, net /P-
- added copper zone on F.Cu, net /P-
- added copper zone on B.Cu, net BAT+
- added copper zone on B.Cu, net BAT1+
- added copper zone on F.Cu, net BAT1+
Other:
- board size 15.4 x 17.7 mm -> 15.3 x 18.2 mm
- board text added: "stiffener polyimide on B.Cu side for all zone on User.eco2 layer"
- board text added: "stiffener polyimide on F.Cu side for all zone on User.eco1 layer"
