File: Hardware/aux_flex_pcb/aux_flex_pcb.kicad_sch (KiCad schematic)
At the start: 17 parts, among them U1 STM32L432KCUx

Commit message: up
Parts:
- removed C10, C13, C27, C8: 100n, v9footprint:C_0201_0603Metric_Pad0.64x0.40mm_HandSolder, symbol Device:C_Small
- removed C15: 10n, v9footprint:C_0201_0603Metric_Pad0.64x0.40mm_HandSolder, symbol Device:C_Small
- removed C16: 1u, v9footprint:C_0201_0603Metric_Pad0.64x0.40mm_HandSolder, symbol Device:C_Small
- removed C19: 4.7u, v9footprint:C_0402_1005Metric, symbol Device:C_Small
- removed LEDBLUE1: 150040BS73240, v9footprint:LED_0402_1005Metric, symbol Device:LED_Small
- removed LEDGREEN1: 150040GS73240, v9footprint:LED_0402_1005Metric, symbol Device:LED_Small
- removed R1, R2: 510R, v9footprint:R_0201_0603Metric_Pad0.64x0.40mm_HandSolder, symbol Device:R_Small
- removed R10, R16: 470k, v9footprint:R_0201_0603Metric_Pad0.64x0.40mm_HandSolder, symbol Device:R_Small
- removed S2: KXT341LHS, v9footprint:KXT341LHS, symbol samacsys:KXT341LHS
- removed TP3: SWCLK, v9footprint:pad_0.7mm, symbol Connector:TestPoint
- removed TP4: SWDIO, v9footprint:pad_0.7mm, symbol Connector:TestPoint
- removed U1: STM32L432KCUx, v9footprint:QFN-32-1EP_5x5mm_P0.5mm_EP3.45x3.45mm, symbol MCU_ST_STM32L4:STM32L432KCUx
- added C14: 100n, v9footprint:C_0201_0603Metric_Pad0.64x0.40mm_HandSolder, symbol Device:C_Small
- added J2: 503548-0622, v9footprint:5035480622, symbol samacsys2:503548-0622
- added R19, R3: 470k, v9footprint:R_0201_0603Metric_Pad0.64x0.40mm_HandSolder, symbol Device:R_Small
- added TP1, TP2: TestPoint, v9footprint:BAT_PAD_1mm, symbol Connector:TestPoint
Connections:
- net BAT+: now also TP2.1
- net GND: now also C14.2, J2.10, J2.3, J2.7, J2.8, J2.9, R19.1, TP1.1
- net GPIO_SUP: now also J2.4
- net OLED_SCL: now also J2.5
- net OLED_SDA: now also J2.2
- net USB_DETECT: now also C14.1, R19.2, R3.1
- new net 3.3V_AUX: J2.1, J2.6
- new net vusb: R3.2
- no-connect marks 4 -> 0
Other:
- removed sheet BTN_CONN
- removed sheet POWER
- removed sheet Peripherial
- note removed: "STM32L432"
- note removed: "wakeup gpio PA0, PC13, PE6, PA2, PC5"

Commit message: up
Parts:
- added J1: 503552-0622, samacsys2:5035520622, symbol samacsys2:503552-0622
- C14: footprint v9footprint:C_0201_0603Metric_Pad0.64x0.40mm_HandSolder -> Capacitor_SMD:C_0201_0603Metric_Pad0.64x0.40mm_HandSolder
- J2: footprint v9footprint:5035480622 -> samacsys2:5035480622
- R19, R3: footprint v9footprint:R_0201_0603Metric_Pad0.64x0.40mm_HandSolder -> Resistor_SMD:R_0201_0603Metric_Pad0.64x0.40mm_HandSolder
- TP1, TP2: footprint v9footprint:BAT_PAD_1mm -> samacsys2:1mm_circle
Connections:
- net 3.3V_AUX: now also J1.1, J1.6
- net GND: now also J1.4, J1.MP1, J1.MP2, J1.MP3, J1.MP4
- new net exti: J1.3
- new net i2c_scl: J1.2
- new net i2c_sda: J1.5

Commit message: up
Parts:
- removed C14: 100n, Capacitor_SMD:C_0201_0603Metric_Pad0.64x0.40mm_HandSolder, symbol Device:C_Small
- removed J2: 503548-0622, samacsys2:5035480622, symbol samacsys2:503548-0622
- removed R3: 470k, Resistor_SMD:R_0201_0603Metric_Pad0.64x0.40mm_HandSolder, symbol Device:R_Small
- added C15, C16, C17, C18: 100n, Capacitor_SMD:C_0201_0603Metric_Pad0.64x0.40mm_HandSolder, symbol Device:C_Small
- added IC1: ICM-42688-P, IIM42352, symbol samacsys:ICM-42688-P
- added R20: 2.2k, Resistor_SMD:R_0201_0603Metric_Pad0.64x0.40mm_HandSolder, symbol Device:R_Small
- added U1: BMP581, BMP581, symbol samacsys:BMP581
- R19: value 470k -> 2.2k
Connections:
- net USB_DETECT is gone; now on net i2c_sda: R19.2
- net 3.3V_AUX: now also R19.1, C15.1, C16.1, C17.1, C18.1, IC1.5 (VDDIO), IC1.8 (VDD), R20.1, U1.1 (VDDIO), U1.10 (VDD)
- net GND: now also C15.2, C16.2, C17.2, C18.2, IC1.6 (GND), U1.3 (VSS_1), U1.8 (VSS_2), U1.9 (VSS_3); no longer R19.1, TP1.1
- net exti: now also IC1.4 (INT1_/_INT)
- net i2c_scl: now also IC1.13 (AP_SCL_/_AP_SCLK), R20.2, U1.2 (SCK)
- net i2c_sda: now also IC1.14 (AP_SDA_/_AP_SDIO_/_AP_SDI), U1.4 (SDI)
- net BAT+: no longer names the net of TP2.1
- no-connect marks 0 -> 10
Other:
- moved on the sheet: J1, R19, TP2

Commit message: up
Parts:
- removed C15, C16, C17, C18: 100n, Capacitor_SMD:C_0201_0603Metric_Pad0.64x0.40mm_HandSolder, symbol Device:C_Small
- removed IC1: ICM-42688-P, IIM42352, symbol samacsys:ICM-42688-P
- removed J1: 503552-0622, samacsys2:5035520622, symbol samacsys2:503552-0622
- removed R19, R20: 2.2k, Resistor_SMD:R_0201_0603Metric_Pad0.64x0.40mm_HandSolder, symbol Device:R_Small
- removed U1: BMP581, BMP581, symbol samacsys:BMP581
- added ANT1: 2450AT14A0100001T, samacsys2:2450AT14A0100001T, symbol samacsys2:2450AT14A0100001T
- added C19, C25: 100n, Capacitor_SMD:C_0201_0603Metric_Pad0.64x0.40mm_HandSolder, symbol Device:C_Small
- added C21, C26, C27: 1u, Capacitor_SMD:C_0201_0603Metric_Pad0.64x0.40mm_HandSolder, symbol Device:C_Small
- added C22, C23: 3.3nF, Capacitor_SMD:C_0201_0603Metric_Pad0.64x0.40mm_HandSolder, symbol Device:C_Small
- added IC2: XB5353A, samacsys2:SOT95P280X125-5N, symbol samacsys2:XB5353A
- added J2, J3: BM29B-2DP_2-0.35V_53_, samacsys2:BM29B2DP2035V53, symbol samacsys2:BM29B-2DP_2-0.35V_53_
- added J4: 503552-0622, samacsys2:5035520622, symbol samacsys2:503552-0622
- added L2: 1.8nH, Inductor_SMD:L_0201_0603Metric_Pad0.64x0.40mm_HandSolder, symbol Device:L_Small
- added R21: 100R, Resistor_SMD:R_0201_0603Metric_Pad0.64x0.40mm_HandSolder, symbol Device:R_Small
- added R22: 100k, Resistor_SMD:R_0201_0603Metric_Pad0.64x0.40mm_HandSolder, symbol Device:R_Small
- added TP3: bat-, symbol Connector:TestPoint
- added TP4: bat+, symbol Connector:TestPoint
- added TP5: gnd, samacsys2:1mm_circle, symbol Connector:TestPoint
- added TP6: swdio, samacsys2:1mm_circle, symbol Connector:TestPoint
- added TP7: swclk, samacsys2:1mm_circle, symbol Connector:TestPoint
- added TP8: rst, samacsys2:1mm_circle, symbol Connector:TestPoint
- added U1: ldln025pu, samacsys:ldln025pu, symbol samacsys:ldln025pu
- added U2: DA14531-00000FX2, samacsys2:FCGQFN24_2.2X3.0_REN, symbol samacsys2:DA14531-00000FX2
- added Y1: 830108254201, samacsys2:830108254201, symbol samacsys2:830108254201
- TP1: value TestPoint -> bat-; footprint samacsys2:1mm_circle -> (none)
- TP2: value TestPoint -> bat+; footprint samacsys2:1mm_circle -> (none)
Connections:
- net 3.3V_AUX: now also C27.1, J4.1, J4.6, U1.4 (VIN)
- net GND: now also C21.2, C22.2, C23.2, C25.2, C26.2, C27.2, IC2.4 (VM_1), IC2.5 (VM_2), J2.1, J2.2, J3.1, J3.2, J4.4, J4.MP1, J4.MP2, J4.MP3, J4.MP4, R22.1, TP3.1, TP5.1, U1.2 (GND), U2.18 (RFIOm), U2.19 (GNDRF1), U2.2 (GNDRF2), U2.20 (GND), U2.21 (GND_DCDC), U2.23 (VSS), Y1.2 (GND(LID))
- net exti: now also J4.3, R22.2, U1.3 (EN)
- net P-: now reaches TP1.1
- net P-: now also C19.2, IC2.2 (GND)
- net BAT+: now reaches TP2.1
- net BAT+: now also J2.5, J2.6, J3.5, J3.6, R21.1, TP4.1
- new net: C19.1, IC2.3 (VDD), R21.2
- new net: U2.3 (XTAL32Mp), Y1.3 (CRYSTAL_2)
- new net: U2.4 (XTAL32Mm), Y1.1 (CRYSTAL_1)
- new net: C21.1, C25.1, C26.1, U1.1 (VOUT), U2.5 (VBAT_LOW), U2.7 (VBAT_HIGH)
- new net: ANT1.1 (FEED), C23.1, L2.2
- new net ADC_SUP: J2.3, J2.4
- new net RF: C22.1, L2.1, U2.1 (RFIOp)
- new net SWCLK: TP7.1, U2.12 (P0_2)
- new net SWDIO: TP6.1, U2.9 (P0_10)
- new net rx_sup: J4.5, TP8.1, U2.10 (RST/P0_0)
- new net tx_sup: J4.2, U2.11 (P0_1)
- no-connect marks 10 -> 12
Other:
- note added: "BAT(No IC)"
- note added: "BAT(Protection IC)"
- note added: "rx on p0.7"

Commit message: up
Parts:
- removed ANT1: 2450AT14A0100001T, samacsys2:2450AT14A0100001T, symbol samacsys2:2450AT14A0100001T
Connections:
- net at U2.3 (XTAL32Mp): now also Y1.1 (CRYSTAL_1); no longer Y1.3 (CRYSTAL_2)
- net at U2.4 (XTAL32Mm): now also Y1.3 (CRYSTAL_2); no longer Y1.1 (CRYSTAL_1)
- no-connect marks 12 -> 13
Other:
- moved on the sheet: Y1

Commit message: up
Parts:
- removed TP1, TP3: bat-, symbol Connector:TestPoint
- removed TP2, TP4: bat+, symbol Connector:TestPoint
- removed TP5: gnd, samacsys2:1mm_circle, symbol Connector:TestPoint
Connections:
- net exti is gone; now on net P-: J4.3, R22.2, U1.3 (EN)
- net BAT+: no longer J3.5, J3.6
- net ADC_SUP: no longer names the net of J2.3
- net ADC_SUP: no longer J2.4
- new net BAT1+: J3.5, J3.6
- no-connect marks 13 -> 15
