File: Hardware/hardware v9/untitled.kicad_sch (KiCad schematic)
At the start: 16 parts, among them IC5 LTC4065EDC#TRMPBF, U2 ldln025pu, U3 ldln025pu, U5 ldln025pu

Commit message: up
Parts:
- C1, C2, C29, C3, C4, C5, C6: footprint v9footprint:C_0201_0603Metric_Pad0.64x0.40mm_HandSolder -> v9footprintlocal:C_0201_0603Metric_Pad0.64x0.40mm_HandSolder
- IC5: footprint v9footprint:SON50P200X200X80-7N-D -> v9footprintlocal:SON50P200X200X80-7N-D
- LEDRED1: footprint v9footprint:LED_0402_1005Metric -> v9footprintlocal:LED_0402_1005Metric
- R17, R21, R27, R4: footprint v9footprint:R_0201_0603Metric_Pad0.64x0.40mm_HandSolder -> v9footprintlocal:R_0201_0603Metric_Pad0.64x0.40mm_HandSolder
- U2, U3, U5: footprint v9footprint:ldln025pu -> v9footprintlocal:ldln025pu
Changed lines of the file:
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@@
 			)
 		)
-		(property "Footprint" "v9footprint:R_0201_0603Metric_Pad0.64x0.40mm_HandSolder"
+		(property "Footprint" "v9footprintlocal:R_0201_0603Metric_Pad0.64x0.40mm_HandSolder"
 			(at 207.01 106.68 0)
 			(hide yes)
@@
 			)
 		)
-		(property "Footprint" "v9footprint:R_0201_0603Metric_Pad0.64x0.40mm_HandSolder"
+		(property "Footprint" "v9footprintlocal:R_0201_0603Metric_Pad0.64x0.40mm_HandSolder"
 			(at 38.1 143.51 0)
 			(hide yes)
@@
 			)
 		)
-		(property "Footprint" "v9footprint:ldln025pu"
+		(property "Footprint" "v9footprintlocal:ldln025pu"
 			(at 216.154 44.45 0)
 			(hide yes)
@@
 			)
 		)
-		(property "Footprint" "v9footprint:R_0201_0603Metric_Pad0.64x0.40mm_HandSolder"
+		(property "Footprint" "v9footprintlocal:R_0201_0603Metric_Pad0.64x0.40mm_HandSolder"
 			(at 205.74 64.77 0)
 			(hide yes)
@@
 			)
 		)
-		(property "Footprint" "v9footprint:C_0201_0603Metric_Pad0.64x0.40mm_HandSolder"
+		(property "Footprint" "v9footprintlocal:C_0201_0603Metric_Pad0.64x0.40mm_HandSolder"
 			(at 191.4652 60.96 0)
 			(hide yes)
@@
 			)
 		)
-		(property "Footprint" "v9footprint:C_0201_0603Metric_Pad0.64x0.40mm_HandSolder"
+		(property "Footprint" "v9footprintlocal:C_0201_0603Metric_Pad0.64x0.40mm_HandSolder"
 			(at 192.7352 102.87 0)
 			(hide yes)
@@
 			)
 		)
-		(property "Footprint" "v9footprint:ldln025pu"
+		(property "Footprint" "v9footprintlocal:ldln025pu"
 			(at 90.424 41.91 0)
 			(hide yes)
@@
 			)
 		)
-		(property "Footprint" "v9footprint:C_0201_0603Metric_Pad0.64x0.40mm_HandSolder"
+		(property "Footprint" "v9footprintlocal:C_0201_0603Metric_Pad0.64x0.40mm_HandSolder"
 			(at 52.07 54.61 0)
 			(hide yes)
@@
 			)
 		)
-		(property "Footprint" "v9footprint:LED_0402_1005Metric"
+		(property "Footprint" "v9footprintlocal:LED_0402_1005Metric"
 			(at 49.53 143.51 90)
 			(hide yes)
@@
 			)
 		)
-		(property "Footprint" "v9footprint:C_0201_0603Metric_Pad0.64x0.40mm_HandSolder"
+		(property "Footprint" "v9footprintlocal:C_0201_0603Metric_Pad0.64x0.40mm_HandSolder"
 			(at 242.2652 102.87 0)
 			(hide yes)
@@
 			)
 		)
-		(property "Footprint" "v9footprint:C_0201_0603Metric_Pad0.64x0.40mm_HandSolder"
+		(property "Footprint" "v9footprintlocal:C_0201_0603Metric_Pad0.64x0.40mm_HandSolder"
 			(at 92.71 153.67 0)
 			(hide yes)
@@
 			)
 		)
-		(property "Footprint" "v9footprint:R_0201_0603Metric_Pad0.64x0.40mm_HandSolder"
+		(property "Footprint" "v9footprintlocal:R_0201_0603Metric_Pad0.64x0.40mm_HandSolder"
 			(at 92.71 140.97 0)
 			(hide yes)
@@
 			)
 		)
-		(property "Footprint" "v9footprint:C_0201_0603Metric_Pad0.64x0.40mm_HandSolder"
+		(property "Footprint" "v9footprintlocal:C_0201_0603Metric_Pad0.64x0.40mm_HandSolder"
 			(at 108.9152 58.42 0)
 			(hide yes)
@@
 			)
 		)
-		(property "Footprint" "v9footprint:ldln025pu"
+		(property "Footprint" "v9footprintlocal:ldln025pu"
 			(at 217.424 86.36 0)
 			(hide yes)
@@
 			)
 		)
-		(property "Footprint" "v9footprint:C_0201_0603Metric_Pad0.64x0.40mm_HandSolder"
+		(property "Footprint" "v9footprintlocal:C_0201_0603Metric_Pad0.64x0.40mm_HandSolder"
 			(at 240.9952 60.96 0)
 			(hide yes)
@@
 			)
 		)
-		(property "Footprint" "v9footprint:SON50P200X200X80-7N-D"
+		(property "Footprint" "v9footprintlocal:SON50P200X200X80-7N-D"
 			(at 86.36 235.89 0)
 			(hide yes)
