File: Hardware/hardware v9/hardware_V9.kicad_sch (KiCad schematic)
At the start: 17 parts, among them U1 STM32L432KCUx

Commit message: up
Other:
- moved on the sheet: TP3, TP4
Changed lines of the file:
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@@
 	(wire
 		(pts
-			(xy 120.65 196.85) (xy 120.65 195.58)
+			(xy 219.71 125.73) (xy 219.71 124.46)
 		)
 		(stroke
@@
 	(wire
 		(pts
-			(xy 107.95 196.85) (xy 107.95 195.58)
+			(xy 207.01 125.73) (xy 207.01 124.46)
 		)
 		(stroke
@@
 	)
 	(label "SWCLK"
-		(at 107.95 196.85 270)
+		(at 207.01 125.73 270)
 		(effects
 			(font
@@
 	)
 	(label "SWDIO"
-		(at 120.65 196.85 270)
+		(at 219.71 125.73 270)
 		(effects
 			(font
@@
 	(symbol
 		(lib_id "Connector:TestPoint")
-		(at 120.65 195.58 0)
+		(at 219.71 124.46 0)
 		(unit 1)
 		(body_style 1)
@@
 		(fields_autoplaced yes)
 		(property "Reference" "TP4"
-			(at 123.19 191.0079 0)
+			(at 222.25 119.8879 0)
 			(show_name no)
 			(do_not_autoplace no)
@@
 		)
 		(property "Value" "SWDIO"
-			(at 123.19 193.5479 0)
+			(at 222.25 122.4279 0)
 			(show_name no)
 			(do_not_autoplace no)
@@
 		)
 		(property "Footprint" "v9footprint:pad_0.7mm"
-			(at 125.73 195.58 0)
+			(at 224.79 124.46 0)
 			(hide yes)
 			(show_name no)
@@
 		)
 		(property "Datasheet" ""
-			(at 125.73 195.58 0)
+			(at 224.79 124.46 0)
 			(hide yes)
 			(show_name no)
@@
 		)
 		(property "Description" "test point"
-			(at 120.65 195.58 0)
+			(at 219.71 124.46 0)
 			(hide yes)
 			(show_name no)
@@
 	(symbol
 		(lib_id "Connector:TestPoint")
-		(at 107.95 195.58 0)
+		(at 207.01 124.46 0)
 		(unit 1)
 		(body_style 1)
@@
 		(fields_autoplaced yes)
 		(property "Reference" "TP3"
-			(at 110.49 191.0079 0)
+			(at 209.55 119.8879 0)
 			(show_name no)
 			(do_not_autoplace no)
@@
 		)
 		(property "Value" "SWCLK"
-			(at 110.49 193.5479 0)
+			(at 209.55 122.4279 0)
 			(show_name no)
 			(do_not_autoplace no)
@@
 		)
 		(property "Footprint" "v9footprint:pad_0.7mm"
-			(at 113.03 195.58 0)
+			(at 212.09 124.46 0)
 			(hide yes)
 			(show_name no)
@@
 		)
 		(property "Datasheet" ""
-			(at 113.03 195.58 0)
+			(at 212.09 124.46 0)
 			(hide yes)
 			(show_name no)
@@
 		)
 		(property "Description" "test point"
-			(at 107.95 195.58 0)
-			(hide yes)
-			(show_name no)
+			(at 207.01 124.46 0)
+			(hide yes)
+			(show_name no)

Commit message: up
Parts:
- C10, C13, C15, C16, C27, C8: footprint v9footprint:C_0201_0603Metric_Pad0.64x0.40mm_HandSolder -> v9footprintlocal:C_0201_0603Metric_Pad0.64x0.40mm_HandSolder
- C19: footprint v9footprint:C_0402_1005Metric -> v9footprintlocal:C_0402_1005Metric
- LEDBLUE1, LEDGREEN1: footprint v9footprint:LED_0402_1005Metric -> v9footprintlocal:LED_0402_1005Metric
- R1, R10, R16, R2: footprint v9footprint:R_0201_0603Metric_Pad0.64x0.40mm_HandSolder -> v9footprintlocal:R_0201_0603Metric_Pad0.64x0.40mm_HandSolder
- S2: footprint v9footprint:KXT341LHS -> v9footprintlocal:KXT341LHS
- TP3, TP4: footprint v9footprint:pad_0.7mm -> v9footprintlocal:pad_0.7mm
- U1: footprint v9footprint:QFN-32-1EP_5x5mm_P0.5mm_EP3.45x3.45mm -> v9footprintlocal:QFN-32-1EP_5x5mm_P0.5mm_EP3.45x3.45mm
Connections:
- net BAT_SENS: now reaches U1.30 (PB7)
- no-connect marks 4 -> 3
Other:
- sheet BTN_CONN ports: added bat_sens; removed none
Changed lines of the file:
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@@
 	)
 	(no_connect
-		(at 125.73 109.22)
-	)
-	(no_connect
 		(at 125.73 88.9)
 	)
@@
 	(wire
 		(pts
+			(xy 326.39 148.59) (xy 331.47 148.59)
+		)
+		(stroke
+			(width 0)
+			(type default)
+		)
+	)
+	(wire
+		(pts
 			(xy 138.43 41.91) (xy 143.51 41.91)
 		)
@@
 		)
 	)
+	(label "BAT_SENS"
+		(at 326.39 148.59 180)
+		(effects
+			(font
+				(size 1.27 1.27)
+			)
+			(justify right bottom)
+		)
+	)
 	(label "GPS_TX"
 		(at 328.93 33.02 180)
@@
 		)
 	)
+	(label "BAT_SENS"
+		(at 125.73 109.22 180)
+		(effects
+			(font
+				(size 1.27 1.27)
+			)
+			(justify right bottom)
+		)
+	)
 	(label "USB_DETECT"
 		(at 153.67 96.52 0)
@@
 			)
 		)
-		(property "Footprint" "v9footprint:C_0201_0603Metric_Pad0.64x0.40mm_HandSolder"
+		(property "Footprint" "v9footprintlocal:C_0201_0603Metric_Pad0.64x0.40mm_HandSolder"
 			(at 116.84 44.45 0)
 			(hide yes)
@@
 			)
 		)
-		(property "Footprint" "v9footprint:KXT341LHS"
+		(property "Footprint" "v9footprintlocal:KXT341LHS"
 			(at 74.93 155.88 0)
 			(hide yes)
@@
 			)
 		)
-		(property "Footprint" "v9footprint:C_0201_0603Metric_Pad0.64x0.40mm_HandSolder"
+		(property "Footprint" "v9footprintlocal:C_0201_0603Metric_Pad0.64x0.40mm_HandSolder"
 			(at 119.38 68.58 0)
 			(hide yes)
@@
 			)
 		)
-		(property "Footprint" "v9footprint:QFN-32-1EP_5x5mm_P0.5mm_EP3.45x3.45mm"
+		(property "Footprint" "v9footprintlocal:QFN-32-1EP_5x5mm_P0.5mm_EP3.45x3.45mm"
 			(at 128.27 119.38 0)
 			(hide yes)
@@
 			)
 		)
-		(property "Footprint" "v9footprint:R_0201_0603Metric_Pad0.64x0.40mm_HandSolder"
+		(property "Footprint" "v9footprintlocal:R_0201_0603Metric_Pad0.64x0.40mm_HandSolder"
 			(at 208.28 74.93 0)
 			(hide yes)
@@
 			)
 		)
-		(property "Footprint" "v9footprint:R_0201_0603Metric_Pad0.64x0.40mm_HandSolder"
+		(property "Footprint" "v9footprintlocal:R_0201_0603Metric_Pad0.64x0.40mm_HandSolder"
 			(at 107.95 116.84 0)
 			(hide yes)
@@
 			)
 		)
-		(property "Footprint" "v9footprint:C_0201_0603Metric_Pad0.64x0.40mm_HandSolder"
+		(property "Footprint" "v9footprintlocal:C_0201_0603Metric_Pad0.64x0.40mm_HandSolder"
 			(at 130.81 44.45 0)
 			(hide yes)
@@
 			)
 		)
-		(property "Footprint" "v9footprint:R_0201_0603Metric_Pad0.64x0.40mm_HandSolder"
+		(property "Footprint" "v9footprintlocal:R_0201_0603Metric_Pad0.64x0.40mm_HandSolder"
 			(at 199.39 67.31 0)
 			(hide yes)
@@
 			)
 		)
-		(property "Footprint" "v9footprint:R_0201_0603Metric_Pad0.64x0.40mm_HandSolder"
+		(property "Footprint" "v9footprintlocal:R_0201_0603Metric_Pad0.64x0.40mm_HandSolder"
 			(at 107.95 107.95 0)
 			(hide yes)
@@
 			)
 		)
-		(property "Footprint" "v9footprint:C_0201_0603Metric_Pad0.64x0.40mm_HandSolder"
+		(property "Footprint" "v9footprintlocal:C_0201_0603Metric_Pad0.64x0.40mm_HandSolder"
 			(at 199.39 74.93 0)
 			(hide yes)
@@
 			)
 		)
-		(property "Footprint" "v9footprint:C_0201_0603Metric_Pad0.64x0.40mm_HandSolder"
+		(property "Footprint" "v9footprintlocal:C_0201_0603Metric_Pad0.64x0.40mm_HandSolder"
 			(at 105.41 44.45 0)
 			(hide yes)
@@
 			)
 		)
-		(property "Footprint" "v9footprint:pad_0.7mm"
+		(property "Footprint" "v9footprintlocal:pad_0.7mm"
 			(at 224.79 124.46 0)
 			(hide yes)
@@
 			)
 		)
-		(property "Footprint" "v9footprint:C_0201_0603Metric_Pad0.64x0.40mm_HandSolder"
+		(property "Footprint" "v9footprintlocal:C_0201_0603Metric_Pad0.64x0.40mm_HandSolder"
 			(at 138.43 44.45 0)
 			(hide yes)
@@
 			)
 		)
-		(property "Footprint" "v9footprint:LED_0402_1005Metric"
+		(property "Footprint" "v9footprintlocal:LED_0402_1005Metric"
 			(at 93.98 107.95 90)
 			(hide yes)
@@
 			)
 		)
-		(property "Footprint" "v9footprint:C_0402_1005Metric"
+		(property "Footprint" "v9footprintlocal:C_0402_1005Metric"
 			(at 92.71 44.45 0)
 			(hide yes)
@@
 			)
 		)
-		(property "Footprint" "v9footprint:pad_0.7mm"
+		(property "Footprint" "v9footprintlocal:pad_0.7mm"
 			(at 212.09 124.46 0)
 			(hide yes)
@@
 			)
 		)
-		(property "Footprint" "v9footprint:LED_0402_1005Metric"
+		(property "Footprint" "v9footprintlocal:LED_0402_1005Metric"
 			(at 93.98 116.84 90)
 			(hide yes)
@@
 			(effects
 				(font
+					(size 1.27 1.27)
+				)
+				(justify left)
+			)
+		)
+		(pin "bat_sens" input
+			(at 331.47 148.59 180)
+			(effects
+				(font

Commit message: up
Connections:
- net GPS_EN: now also U1.3 (PC15); no longer U1.14 (PB0)
- net SD_DET: now also U1.25 (PA15); no longer U1.27 (PB4)
- net at R1.1: now also U1.27 (PB4); no longer U1.28 (PB5)
- net at R2.1: now also U1.28 (PB5); no longer U1.29 (PB6)
- net BAT_SENS renamed RX_SUP
- new net ADC_SUP: U1.14 (PB0)
- new net TX_SUP: U1.29 (PB6)
- no-connect marks 3 -> 1
Other:
- sheet BTN_CONN ports: added rx_sup/sda, tx_sup/scl; removed none
Changed lines of the file:
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@@
 	)
 	(no_connect
-		(at 151.13 114.3)
-	)
-	(no_connect
-		(at 125.73 88.9)
-	)
-	(no_connect
 		(at 125.73 86.36)
 	)
@@
 	(wire
 		(pts
-			(xy 125.73 106.68) (xy 115.57 106.68)
+			(xy 328.93 29.21) (xy 332.74 29.21)
 		)
 		(stroke
@@
 	(wire
 		(pts
-			(xy 121.92 101.6) (xy 125.73 101.6)
+			(xy 140.97 68.58) (xy 144.78 68.58)
 		)
 		(stroke
@@
 	(wire
 		(pts
-			(xy 328.93 29.21) (xy 332.74 29.21)
+			(xy 124.46 106.68) (xy 125.73 106.68)
 		)
 		(stroke
@@
 	(wire
 		(pts
-			(xy 140.97 68.58) (xy 144.78 68.58)
+			(xy 153.67 96.52) (xy 151.13 96.52)
 		)
 		(stroke
@@
 	(wire
 		(pts
-			(xy 153.67 96.52) (xy 151.13 96.52)
+			(xy 121.92 68.58) (xy 124.46 68.58)
 		)
 		(stroke
@@
 	(wire
 		(pts
-			(xy 121.92 68.58) (xy 124.46 68.58)
+			(xy 115.57 104.14) (xy 115.57 116.84)
 		)
 		(stroke
@@
 	(wire
 		(pts
-			(xy 115.57 106.68) (xy 115.57 116.84)
+			(xy 153.67 104.14) (xy 151.13 104.14)
 		)
 		(stroke
@@
 	(wire
 		(pts
-			(xy 153.67 104.14) (xy 151.13 104.14)
+			(xy 115.57 68.58) (xy 116.84 68.58)
 		)
 		(stroke
@@
 	(wire
 		(pts
-			(xy 115.57 68.58) (xy 116.84 68.58)
+			(xy 153.67 114.3) (xy 151.13 114.3)
 		)
 		(stroke
@@
 	(wire
 		(pts
-			(xy 113.03 107.95) (xy 113.03 104.14)
+			(xy 113.03 101.6) (xy 113.03 107.95)
+		)
+		(stroke
+			(width 0)
+			(type default)
+		)
+	)
+	(wire
+		(pts
+			(xy 125.73 104.14) (xy 115.57 104.14)
 		)
 		(stroke
@@
 	(wire
 		(pts
+			(xy 327.66 124.46) (xy 331.47 124.46)
+		)
+		(stroke
+			(width 0)
+			(type default)
+		)
+	)
+	(wire
+		(pts
 			(xy 153.67 88.9) (xy 151.13 88.9)
 		)
@@
 	(wire
 		(pts
+			(xy 327.66 128.27) (xy 331.47 128.27)
+		)
+		(stroke
+			(width 0)
+			(type default)
+		)
+	)
+	(wire
+		(pts
 			(xy 153.67 76.2) (xy 151.13 76.2)
 		)
@@
 	(wire
 		(pts
-			(xy 113.03 104.14) (xy 125.73 104.14)
+			(xy 105.41 116.84) (xy 96.52 116.84)
 		)
 		(stroke
@@
 	(wire
 		(pts
-			(xy 105.41 116.84) (xy 96.52 116.84)
+			(xy 330.2 77.47) (xy 332.74 77.47)
 		)
 		(stroke
@@
 	(wire
 		(pts
-			(xy 330.2 77.47) (xy 332.74 77.47)
+			(xy 151.13 67.31) (xy 144.78 67.31)
 		)
 		(stroke
@@
 	(wire
 		(pts
-			(xy 151.13 67.31) (xy 144.78 67.31)
+			(xy 330.2 66.04) (xy 332.74 66.04)
 		)
 		(stroke
@@
 	(wire
 		(pts
-			(xy 330.2 66.04) (xy 332.74 66.04)
+			(xy 92.71 46.99) (xy 105.41 46.99)
 		)
 		(stroke
@@
 	(wire
 		(pts
-			(xy 92.71 46.99) (xy 105.41 46.99)
+			(xy 153.67 83.82) (xy 151.13 83.82)
 		)
 		(stroke
@@
 	(wire
 		(pts
-			(xy 153.67 83.82) (xy 151.13 83.82)
+			(xy 125.73 101.6) (xy 113.03 101.6)
 		)
 		(stroke
@@
 	(wire
 		(pts
+			(xy 124.46 109.22) (xy 125.73 109.22)
+		)
+		(stroke
+			(width 0)
+			(type default)
+		)
+	)
+	(wire
+		(pts
 			(xy 328.93 161.29) (xy 331.47 161.29)
 		)
@@
 	(wire
 		(pts
+			(xy 121.92 88.9) (xy 125.73 88.9)
+		)
+		(stroke
+			(width 0)
+			(type default)
+		)
+	)
+	(wire
+		(pts
 			(xy 121.92 93.98) (xy 125.73 93.98)
 		)
@@
 		)
 	)
-	(label "SD_DET"
-		(at 121.92 101.6 180)
+	(label "RX_SUP"
+		(at 124.46 109.22 180)
+		(effects
+			(font
+				(size 1.27 1.27)
+			)
+			(justify right bottom)
+		)
+	)
+	(label "RX_SUP"
+		(at 327.66 124.46 180)
 		(effects
 			(font
@@
 		)
 	)
+	(label "SD_DET"
+		(at 153.67 114.3 0)
+		(effects
+			(font
+				(size 1.27 1.27)
+			)
+			(justify left bottom)
+		)
+	)
 	(label "USB_DETECT"
 		(at 327.66 113.03 180)
@@
 		)
 	)
-	(label "BAT_SENS"
-		(at 326.39 148.59 180)
+	(label "GPS_TX"
+		(at 328.93 33.02 180)
 		(effects
 			(font
@@
 		)
 	)
-	(label "GPS_TX"
-		(at 328.93 33.02 180)
+	(label "SWCLK"
+		(at 207.01 125.73 270)
 		(effects
 			(font
@@
 		)
 	)
-	(label "SWCLK"
-		(at 207.01 125.73 270)
+	(label "GPIO_SUP"
+		(at 326.39 144.78 180)
 		(effects
 			(font
@@
 		)
 	)
-	(label "GPIO_SUP"
-		(at 326.39 144.78 180)
+	(label "TX_SUP"
+		(at 327.66 128.27 180)
 		(effects
 			(font
@@
 		)
 	)
-	(label "GPS_EN"
+	(label "ADC_SUP"
+		(at 326.39 148.59 180)
+		(effects
+			(font
+				(size 1.27 1.27)
+			)
+			(justify right bottom)
+		)
+	)
+	(label "ADC_SUP"
 		(at 121.92 93.98 180)
 		(effects
@@
 		)
 	)
-	(label "BAT_SENS"
-		(at 125.73 109.22 180)
-		(effects
-			(font
-				(size 1.27 1.27)
-			)
-			(justify right bottom)
-		)
-	)
 	(label "USB_DETECT"
 		(at 153.67 96.52 0)
@@
 		)
 	)
+	(label "TX_SUP"
+		(at 124.46 106.68 180)
+		(effects
+			(font
+				(size 1.27 1.27)
+			)
+			(justify right bottom)
+		)
+	)
 	(label "SPI_MISO"
 		(at 153.67 91.44 0)
@@
 		)
 	)
+	(label "GPS_EN"
+		(at 121.92 88.9 180)
+		(effects
+			(font
+				(size 1.27 1.27)
+			)
+			(justify right bottom)
+		)
+	)
 	(label "OLED_SCL"
 		(at 327.66 133.35 180)
@@
 			(effects
 				(font
+					(size 1.27 1.27)
+				)
+				(justify left)
+			)
+		)
+		(pin "rx_sup{slash}sda" input
+			(at 331.47 124.46 180)
+			(effects
+				(font
+					(size 1.27 1.27)
+				)
+				(justify left)
+			)
+		)
+		(pin "tx_sup{slash}scl" input
+			(at 331.47 128.27 180)
+			(effects
+				(font
