File: Hardware/hardware v9/BTN_CONN.kicad_sch (KiCad schematic)
At the start: 16 parts, among them J2 503548-0622, J3 USB4110-GF-A

Commit message: up
Other:
- note added: "PULL DOWN FOR BOOT0 BE AWARE IN THE SOFTWARE"
- moved on the sheet: C20, C7, R7, R9, S1, S3, TP1, TP2

Commit message: up
Parts:
- removed TP1, TP2: TestPoint, v9footprint:BAT_PAD_1mm, symbol Connector:TestPoint
- added J4: BM29B0.6-2DS_2-0.35V_53_, BM29B062DS2035V53, symbol samacsys2:BM29B0.6-2DS_2-0.35V_53_
- C14, C20, C7: footprint v9footprint:C_0201_0603Metric_Pad0.64x0.40mm_HandSolder -> v9footprintlocal:C_0201_0603Metric_Pad0.64x0.40mm_HandSolder
- J2: footprint v9footprint:5035480622 -> v9footprintlocal:5035480622
- J3: footprint v9footprint:USB4110GFA -> v9footprintlocal:USB4110GFA
- R19, R22, R23, R3, R7, R9: footprint v9footprint:R_0201_0603Metric_Pad0.64x0.40mm_HandSolder -> v9footprintlocal:R_0201_0603Metric_Pad0.64x0.40mm_HandSolder
- S1, S3: footprint v9footprint:PTS845VM20PSMTR4LFS -> v9footprintlocal:PTS845VM20PSMTR4LFS
- U4: footprint v9footprint:ssd1306_5point -> v9footprintlocal:ssd1306_5point
Connections:
- net BAT+: now also J4.1, J4.2
- net GND: now also J4.5, J4.6, J4.MP1, J4.MP2, J4.MP3, J4.MP4
- new net bat_sens: J4.3, J4.4

Commit message: up
Connections:
- net BAT+: now also J4.MP1, J4.MP2
- net GND: no longer J4.MP1, J4.MP2
- net OLED_SCL: no longer J2.5
- net OLED_SDA: no longer J2.2
- new net rx_sup/sda: J2.5
- new net tx_sup/scl: J2.2

Commit message: up
Parts:
- J4: footprint BM29B062DS2035V53 -> samacsys2:BM29B062DS2035V53
Changed lines of the file:
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@@
 			)
 		)
-		(property "Footprint" "BM29B062DS2035V53"
+		(property "Footprint" "samacsys2:BM29B062DS2035V53"
 			(at 111.76 216.84 0)
 			(hide yes)
