File: Hardware/hardware v9/hardware_V9.kicad_pcb (KiCad board)
At the start: 6 copper layers, 22.7 x 19 mm, 63 parts, among them IC5 LTC4065EDC#TRMPBF, J1 Micro_SD_Card_Det2, J2 503548-0622, J3 USB4110-GF-A, U1 STM32L432KCUx, U2 ldln025pu, U3 ldln025pu, U5 ldln025pu

Commit message: up
Parts:
- C1, C10, C11, C12, C13, C14, C15, C16, C17, C2, C20, C27, C29, C3, C4, C5, C6, C7, C8: footprint v9footprint:C_0201_0603Metric_Pad0.64x0.40mm_HandSolder -> v9footprintlocal:C_0201_0603Metric_Pad0.64x0.40mm_HandSolder
- C19, C21: footprint v9footprint:C_0402_1005Metric -> v9footprintlocal:C_0402_1005Metric
- IC5: footprint v9footprint:SON50P200X200X80-7N-D -> v9footprintlocal:SON50P200X200X80-7N-D
- J1: footprint v9footprint:microSD_HC_Molex_104031-0811 -> v9footprintlocal:microSD_HC_Molex_104031-0811
- J2: footprint v9footprint:5035480622 -> v9footprintlocal:5035480622
- J3: footprint v9footprint:USB4110GFA -> v9footprintlocal:USB4110GFA
- LEDBLUE1, LEDGREEN1, LEDRED1: footprint v9footprint:LED_0402_1005Metric -> v9footprintlocal:LED_0402_1005Metric
- PA1010D1: footprint v9footprint:PA1010D -> v9footprintlocal:PA1010D
- R1, R10, R13, R14, R15, R16, R17, R18, R19, R2, R20, R21, R22, R23, R24, R25, R26, R27, R3, R4, R7, R9: footprint v9footprint:R_0201_0603Metric_Pad0.64x0.40mm_HandSolder -> v9footprintlocal:R_0201_0603Metric_Pad0.64x0.40mm_HandSolder
- S1, S3: footprint v9footprint:PTS845VM20PSMTR4LFS -> v9footprintlocal:PTS845VM20PSMTR4LFS
- S2: footprint v9footprint:KXT341LHS -> v9footprintlocal:KXT341LHS
- TP1, TP2: footprint v9footprint:BAT_PAD_1mm -> v9footprintlocal:BAT_PAD_1mm
- TP3, TP4: footprint v9footprint:pad_0.7mm -> v9footprintlocal:pad_0.7mm
- U1: footprint v9footprint:QFN-32-1EP_5x5mm_P0.5mm_EP3.45x3.45mm -> v9footprintlocal:QFN-32-1EP_5x5mm_P0.5mm_EP3.45x3.45mm
- U2, U3, U5: footprint v9footprint:ldln025pu -> v9footprintlocal:ldln025pu
- U4: footprint v9footprint:ssd1306_5point -> v9footprintlocal:ssd1306_5point

Commit message: up
Parts:
- removed TP1, TP2: TestPoint, v9footprintlocal:BAT_PAD_1mm
- added J4: BM29B0.6-2DS_2-0.35V_53_, samacsys2:BM29B062DS2035V53, F.Cu at (107.7, 107.4)
- C21: footprint v9footprintlocal:C_0402_1005Metric -> v9footprintlocal:LED_0402_1005Metric
- moved S1 0.12 mm to (107.7, 93.5)
Connections:
- U1 pad 30: unconnected-(U1-PB7-Pad30) -> /BAT_SENS
Routing:
- net /BAT_SENS: track 0.00 -> 17.3 mm, vias 0 -> 2
- net GND: vias 72 -> 74
- net BAT+: vias 6 -> 8
- added copper zone on B.Cu, net /SWCLK
- added copper zone on B.Cu, net /SWDIO

Commit message: up
Parts:
- moved C12 4.12 mm to (115.5, 96.7)
- moved TP3 0.65 mm to (94.9, 97.8)
- moved C17 0.30 mm to (115.5, 100.8)
- moved R18 0.30 mm to (115.5, 98.8)
- moved J1 0.25 mm to (108.8, 100.2)
- moved R20 0.20 mm to (115.5, 103.3)
Connections:
- J2 pad 2: /OLED_SDA -> /TX_SUP
- J2 pad 5: /OLED_SCL -> /RX_SUP
- J4 pad 3: /BAT_SENS -> /ADC_SUP
- J4 pad 4: /BAT_SENS -> /ADC_SUP
- J4 pad MP1: GND -> BAT+
- J4 pad MP2: GND -> BAT+
- R1 pad 1: Net-(U1-PB5) -> Net-(U1-PB4)
- R2 pad 1: Net-(U1-PB6) -> Net-(U1-PB5)
- U1 pad 14: /GPS_EN -> /ADC_SUP
- U1 pad 25: unconnected-(U1-PA15-Pad25) -> /SD_DET
- U1 pad 27: /SD_DET -> Net-(U1-PB4)
- U1 pad 29: Net-(U1-PB6) -> /TX_SUP
- U1 pad 3: unconnected-(U1-PC15-Pad3) -> /GPS_EN
- U1 pad 30: /BAT_SENS -> /RX_SUP
Routing:
- net /BAT_SENS: track 17.3 -> 0.00 mm, vias 2 -> 0
- net /ADC_SUP: track 0.00 -> 15.6 mm, vias 0 -> 2
- net /RX_SUP: track 0.00 -> 9.47 mm, vias 0 -> 2
- net /TX_SUP: track 0.00 -> 8.93 mm, vias 0 -> 2
- net vusb: track 9.10 -> 14.9 mm, vias 3 -> 2
- net /GPS_EN: track 12.4 -> 16.0 mm, vias 1 -> 2
- net 3.3V_GPS: track 14.6 -> 11.2 mm
- net /OLED_SCL: track 9.17 -> 5.88 mm, vias 1 -> 0
- net Net-(U1-PB6): track 2.16 -> 0.00 mm
- net /B1: track 22.0 -> 23.6 mm
- net Net-(U1-PB4): track 0.00 -> 1.46 mm
- net /OLED_SDA: track 7.91 -> 6.50 mm, vias 1 -> 0
- net Net-(U1-PB5): track 1.46 -> 2.54 mm
- net /D-: track 7.16 -> 6.08 mm
- net 3.3V_AUX: track 18.1 -> 18.9 mm
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- removed copper zone on In3.Cu, net vusb
Other:
- outline, holes or cut-outs redrawn
- board text added: "V10.0"
- board text removed: "V9.0"
