File: Hardware/custom_10x10mm_m10_gps/custom_gps.kicad_pcb (KiCad board)
At the start: 6 copper layers, 10 x 10 mm, 15 parts, among them IC1 MIA-M10Q-00B, J1 830107834801

Commit message: up
Parts:
- added C10: 1u, Capacitor_SMD:C_0201_0603Metric, F.Cu at (117.0, 89.9)
- added C11: 10u, Capacitor_SMD:C_0402_1005Metric, F.Cu at (119.6, 88.5)
- added C12: 10u, Capacitor_SMD:C_0402_1005Metric, F.Cu at (119.6, 90.5)
- added C7: 4.7u, Capacitor_SMD:C_0402_1005Metric, F.Cu at (119.6, 86.5)
- added C8: 100n, Capacitor_SMD:C_0201_0603Metric, F.Cu at (117.0, 86.4)
- added C9: 1u, Capacitor_SMD:C_0201_0603Metric, F.Cu at (117.0, 88.2)
- added D3: RB521S-30DP-TP, samacsys2:RB521S30DPTP, F.Cu at (120.1, 93.2)
- added R4: 4.7k, Resistor_SMD:R_0201_0603Metric, F.Cu at (117.0, 91.7)
- added R5: 4.7k, Resistor_SMD:R_0201_0603Metric, F.Cu at (117.0, 93.4)
- added R6: 560k, Resistor_SMD:R_0201_0603Metric, F.Cu at (117.0, 95.2)
- added R7: 4.7k, Resistor_SMD:R_0201_0603Metric, F.Cu at (117.0, 96.9)
- added U1: ~, samacsys2:ssd1306_fpc, F.Cu at (132.8, 86.3)
- added U4: ~, samacsys2:ssd1306_5point, F.Cu at (132.6, 90.6)
