File: Hardware/custom_10x10mm_m10_gps/custom_gps.kicad_pcb (KiCad board)
At the start: 6 copper layers, 10 x 10 mm, 28 parts, among them IC1 MIA-M10Q-00B, J1 830107834801

Commit message: up
Parts:
- removed C10, C9: 1u, Capacitor_SMD:C_0201_0603Metric
- removed C11, C12: 10u, Capacitor_SMD:C_0402_1005Metric
- removed C7: 4.7u, Capacitor_SMD:C_0402_1005Metric
- removed C8: 100n, Capacitor_SMD:C_0201_0603Metric
- removed D3: RB521S-30DP-TP, samacsys2:RB521S30DPTP
- removed R4, R5, R7: 4.7k, Resistor_SMD:R_0201_0603Metric
- removed R6: 560k, Resistor_SMD:R_0201_0603Metric
- removed U1: ~, samacsys2:ssd1306_fpc
- removed U4: ~, samacsys2:ssd1306_5point
