File: Hardware/custom_10x10mm_m10_gps/custom_gps.kicad_sch (KiCad schematic)
At the start: 14 parts, among them IC1 MIA-M10Q-00B, J1 830107834801

Commit message: up
Parts:
- Connpa1010d1: value ~ -> (none)
- D1, D2: footprint RCLAMP3521ZATFT -> samacsys:RCLAMP3521ZATFT
Other:
- added sheet ssd1306 (ssd1306.kicad_sch)
