File: Hardware/hardware v11/BTN_CONN.kicad_sch (KiCad schematic)
At the start: 13 parts, among them J2 503548-0622, J3 USB4110-GF-A, J4 BM29B0.6-2DS_2-0.35V_53_

Commit message: up
Parts:
- removed C14: 100n, v9footprintlocal:C_0201_0603Metric_Pad0.64x0.40mm_HandSolder, symbol Device:C_Small
- removed J4: BM29B0.6-2DS_2-0.35V_53_, samacsys2:BM29B062DS2035V53, symbol samacsys2:BM29B0.6-2DS_2-0.35V_53_
- removed R3: 470k, v9footprintlocal:R_0201_0603Metric_Pad0.64x0.40mm_HandSolder, symbol Device:R_Small
- added C9: 100n, v9footprintlocal:C_0201_0603Metric_Pad0.64x0.40mm_HandSolder, symbol Device:C_Small
- added J4: Conn_01x02_MountingPin, Connector_JST:JST_SUR_BM02B-SURS-TF_1x02-1MP_P0.80mm_Vertical, symbol Connector_Generic_MountingPin:Conn_01x02_MountingPin
- added R11, R8: 5.1k, v9footprintlocal:R_0201_0603Metric_Pad0.64x0.40mm_HandSolder, symbol Device:R_Small
- added R12, R24: 470k, v9footprintlocal:R_0201_0603Metric_Pad0.64x0.40mm_HandSolder, symbol Device:R_Small
- J3: footprint v9footprintlocal:USB4110GFA -> Connector_USB:USB_C_Receptacle_GCT_USB4105-xx-A_16P_TopMnt_Horizontal
- R19: Mouser Part Number 603-AC0201FR-07470KL -> 603-AC0201FR-0720KL; Mouser Price/Stock https://www.mouser.fr/ProductDetail/YAGEO/AC0201FR-07470KL?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 -> https://www.mouser.fr/ProductDetail/YAGEO/AC0201FR-0720KL?q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
Connections:
- net BAT+: now also J4.1 (Pin_1)
- net GND: now also J3.SH (MP1), C9.2, J4.2 (Pin_2), J4.MP (MountPin), R11.1, R8.2; no longer J3.MP1, J3.MP2, J3.MP3, J3.MP4, U4.6 (GND)
- net vusb: now also R12.2
- net CC1: no longer names the net of J3.A5 (CC1)
- net CC1: now also R8.1
- net CC2: no longer names the net of J3.B5 (CC2)
- net CC2: now also R11.2
- net USB_DETECT renamed USB_DET
- net USB_DET: now also C9.1, R12.1
- new net: R24.1, U4.6 (SUP_2)
- new net ECRAN_SUP: R24.2
