File: Hardware/hardware v11/hardware_V11.kicad_pcb (KiCad board)
At the start: 6 copper layers, 22.7 x 19 mm, 57 parts, among them IC5 LTC4065EDC#TRMPBF, J1 Micro_SD_Card_Det2, J2 503548-0622, J3 USB4110-GF-A, J4 BM29B0.6-2DS_2-0.35V_53_, U2 ldln025pu, U3 ldln025pu, U5 ldln025pu, U6 STM32G0B1KCUx

Commit message: up
Parts:
- removed S2: KXT341LHS, v9footprintlocal:KXT341LHS
- added C13: 100n, v9footprintlocal:C_0201_0603Metric_Pad0.64x0.40mm_HandSolder, B.Cu at (105.8, 97.9)
- added C15: 100n, v9footprintlocal:C_0201_0603Metric_Pad0.64x0.40mm_HandSolder, B.Cu at (104.6, 97.8)
- added C16: 100n, v9footprintlocal:C_0201_0603Metric_Pad0.64x0.40mm_HandSolder, B.Cu at (103.7, 97.8)
- added C24: 4.7u, v9footprintlocal:C_0402_1005Metric, B.Cu at (105.8, 103.2)
- added C25: 4.7u, v9footprintlocal:C_0402_1005Metric, F.Cu at (114.0, 107.5)
- added C9: 100n, v9footprintlocal:C_0201_0603Metric_Pad0.64x0.40mm_HandSolder, B.Cu at (102.0, 95.0)
- added IC1: DPS368XTSA1, samacsys:DPS368XTSA1, B.Cu at (104.3, 95.8)
- added IC2: ICM-42688-P, samacsys:IIM42352, B.Cu at (104.8, 100.6)
- added IC3: MMC5603NJ, samacsys2:MMC5603NJ, F.Cu at (115.8, 107.7)
- added IC4: TPD2EUSB30ADRTR, samacsys2:SOT35P100X50-3N, F.Cu at (0.97, 0.48)
- added R11: 5.1k, v9footprintlocal:R_0201_0603Metric_Pad0.64x0.40mm_HandSolder, B.Cu at (102.0, 97.1)
- added R12: 470k, v9footprintlocal:R_0201_0603Metric_Pad0.64x0.40mm_HandSolder, B.Cu at (102.0, 96.4)
- added R22: 4.7k, v9footprintlocal:R_0201_0603Metric_Pad0.64x0.40mm_HandSolder, B.Cu at (113.0, 107.2)
- added R23: 4.7k, v9footprintlocal:R_0201_0603Metric_Pad0.64x0.40mm_HandSolder, B.Cu at (113.0, 108.0)
- added R8: 5.1k, v9footprintlocal:R_0201_0603Metric_Pad0.64x0.40mm_HandSolder, B.Cu at (101.8, 101.4)
- added TP5: SWCLK, v9footprintlocal:pad_0.7mm, F.Cu at (95.0, 101.9)
- C1, C3, C5, C6, R14, R15, R26, U3, U5: moved to F.Cu
- C14, C29, IC5, R17, R19, R21, R27, R4: moved to B.Cu
- C21: footprint v9footprintlocal:LED_0402_1005Metric -> v9footprintlocal:C_0402_1005Metric
- J3: footprint v9footprintlocal:USB4110GFA -> Connector_USB:USB_C_Receptacle_GCT_USB4105-xx-A_16P_TopMnt_Horizontal
- J4: value BM29B0.6-2DS_2-0.35V_53_ -> Conn_01x02_MountingPin; footprint samacsys2:BM29B062DS2035V53 -> Connector_JST:JST_SUR_BM02B-SURS-TF_1x02-1MP_P0.80mm_Vertical
- R24: value 0R -> 470k; moved to B.Cu
- R3: value 470k -> 0R
- moved R24 19.6 mm to (95.7, 105.3), turned to 180 degrees
- moved C1 16.3 mm to (113.1, 107.5), turned to 90 degrees
- moved U5 14.3 mm to (111.8, 107.5), turned to 180 degrees
- moved R27 13.3 mm to (107.1, 107.5), turned to 90 degrees
- moved R21 13.2 mm to (110.2, 107.5)
- moved C6 12.8 mm to (110.2, 107.5), turned to -90 degrees
- moved C3 11.9 mm to (106.0, 107.5), turned to 90 degrees
- moved C5 11.6 mm to (109.2, 107.5), turned to -90 degrees
- moved TP3 10.0 mm to (102.2, 96.7)
- moved TP4 9.99 mm to (102.0, 97.8)
- moved C14 9.94 mm to (105.0, 103.2), turned to -90 degrees
- moved U3 9.64 mm to (107.5, 107.4)
- moved R17 8.83 mm to (105.5, 104.5), turned to 0 degrees
- moved J4 8.80 mm to (98.9, 106.9), turned to 180 degrees
- moved R14 8.35 mm to (97.2, 104.2), turned to 90 degrees
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Connections:
- C14 pad 1: /USB_DETECT -> 3.3V_AUX
- C7 pad 1: /SWCLK -> /B1
- J3 pad A5: /PD_CC1 -> Net-(J3-CC1)
- J3 pad B5: /PD_CC2 -> Net-(J3-CC2)
- J4 pad 2: BAT+ -> GND
- PA1010D1 pad 9: Net-(PA1010D1-VBACKUP) -> BAT+
- R1 pad 1: Net-(U6-PB5) -> Net-(U6-PC14)
- R19 pad 2: /USB_DETECT -> /USB_DET
- R2 pad 1: Net-(U6-PB6) -> Net-(U6-PC15)
- R24 pad 1: BAT+ -> Net-(U4-SUP_2)
- R24 pad 2: Net-(PA1010D1-VBACKUP) -> /ECRAN_SUP
- R3 pad 1: /USB_DETECT -> /B1
- R3 pad 2: vusb -> Net-(U6-PA14)
- R7 pad 1: /SWCLK -> /B1
- S1 pad 2: /SWCLK -> /B1
- TP3 pad 1: /SWCLK -> Net-(U6-PA14)
- U4 pad 6: GND -> Net-(U4-SUP_2)
- U6 pad 15: /AUX_EN -> /GPS_EN
- U6 pad 16: /SD_DET -> /AUX_EN
- U6 pad 17: /USB_DETECT -> /SD_DET
- U6 pad 18: /PD_CC1 -> unconnected-(U6-PA8-Pad18)
- U6 pad 19: /PD_CC1 -> /SENSOR_SCL
- U6 pad 2: unconnected-(U6-PC14-Pad2) -> Net-(U6-PC14)
- U6 pad 20: unconnected-(U6-PC6-Pad20) -> /USB_DET
- U6 pad 21: /PD_CC2 -> /SENSOR_SDA
- U6 pad 25: /SWCLK -> Net-(U6-PA14)
- U6 pad 26: /SWCLK -> /B1
- U6 pad 29: Net-(U6-PB5) -> unconnected-(U6-PB5-Pad29)
- U6 pad 3: /GPS_EN -> Net-(U6-PC15)
- U6 pad 30: Net-(U6-PB6) -> /OLED_SCL
- U6 pad 32: /OLED_SCL -> /ECRAN_SUP
Routing:
- net /SENSOR_SDA: track 0.00 -> 31.6 mm, vias 0 -> 3
- net /SENSOR_SCL: track 0.00 -> 30.4 mm, vias 0 -> 3
- net BAT+: track 0.00 -> 19.6 mm, vias 8 -> 9
- net /SWCLK: track 17.2 -> 0.00 mm, vias 1 -> 0
- net Net-(PA1010D1-TX): track 0.00 -> 14.0 mm, vias 0 -> 2
- net 3.3V_AUX: track 18.9 -> 32.8 mm, vias 7 -> 12
- net Net-(PA1010D1-RX): track 0.00 -> 13.5 mm, vias 0 -> 2
- net /SPI_MISO: track 12.2 -> 25.5 mm, vias 0 -> 2
- net /B1: track 0.00 -> 13.2 mm, vias 0 -> 2
- net Net-(PA1010D1-VBACKUP): track 12.5 -> 0.00 mm, vias 2 -> 0
- net /SPI_CS: track 17.9 -> 29.3 mm, vias 1 -> 2
- net /SD_DET: track 2.55 -> 13.5 mm, vias 1 -> 2
- net /ECRAN_SUP: track 0.00 -> 10.8 mm, vias 0 -> 2
- net 3.3V_GPS: track 11.2 -> 1.91 mm, vias 1 -> 4
- net /AUX_EN: track 7.23 -> 16.2 mm, vias 1 -> 2
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- added copper zone on F.Cu, net 3.3V_GPS
- added copper zone on In3.Cu, net 3.3V_GPS
- added copper zone on B.Cu, net vusb
- removed copper zone on B.Cu, net /SWCLK
- removed copper zone on B.Cu, net /SWDIO
- removed copper zone on B.Cu, net 3.3V_GPS
- removed copper zone on F.Cu, net vusb
Other:
- board text added: "V12.0 m.pommery"
- board text removed: "V10.0"
- board text removed: "m.pommery"
