File: Hardware/hardware v11/hardware_V11.kicad_pcb (KiCad board)
At the start: 6 copper layers, 22.7 x 19 mm, 72 parts, among them IC1 DPS368XTSA1, IC2 ICM-42688-P, IC3 MMC5603NJ, IC4 TPD2EUSB30ADRTR, IC5 LTC4065EDC#TRMPBF, J1 Micro_SD_Card_Det2, J2 503548-0622, J3 USB4110-GF-A, J4 Conn_01x02_MountingPin, U2 ldln025pu, U3 ldln025pu, U5 ldln025pu, U6 STM32G0B1KCUx

Commit message: up
Parts:
- removed IC4: TPD2EUSB30ADRTR, samacsys2:SOT35P100X50-3N
