File: Hardware/hardware v11/hardware_V11.kicad_sch (KiCad schematic)
At the start: 14 parts, among them U6 STM32G0B1KCUx

Commit message: up
Parts:
- removed S2: KXT341LHS, v9footprintlocal:KXT341LHS, symbol samacsys:KXT341LHS
- added R3: 0R, v9footprintlocal:R_0201_0603Metric_Pad0.64x0.40mm_HandSolder, symbol Device:R_Small
- added TP5: SWCLK, v9footprintlocal:pad_0.7mm, symbol Connector:TestPoint
Connections:
- net USB_DETECT is gone; now on net SD_DET: U6.17 (PB2)
- net AUX_EN: now also U6.16 (PB1); no longer U6.15 (PB0)
- net GPS_EN: now also U6.15 (PB0); no longer U6.3 (PC15)
- net NRST: now also TP5.1
- net OLED_SCL: now also U6.30 (PB6); no longer U6.32 (PB8)
- net SD_DET: no longer U6.16 (PB1)
- net at R2.1: now also U6.3 (PC15); no longer U6.30 (PB6)
- net at R1.1: now also U6.2 (PC14); no longer U6.29 (PB5)
- net USB_DET: now reaches U6.20 (PC6)
- net PD_CC1: no longer names the net of U6.18 (PA8)
- net PD_CC1: no longer U6.19 (PA9/UCPD1_DBCC1)
- net PD_CC2 renamed SENSOR_SDA
- net SWCLK: no longer names the net of TP3.1, U6.25 (PA14)
- net SWCLK: now also R3.2; no longer U6.26 (PA15)
- new net B1: R3.1, U6.26 (PA15)
- new net ECRAN_SUP: U6.32 (PB8)
- new net SENSOR_SCL: U6.19 (PA9/UCPD1_DBCC1)
Other:
- sheet BTN_CONN ports: added ECRAN_SUP, USB_DET; removed CC1, CC2, USB_DETECT, bat_sens
- sheet POWER ports: added none; removed CH_EN
- sheet Peripherial ports: added SENSOR_SCL, SENSOR_SDA; removed none
- moved on the sheet: LEDBLUE1, LEDGREEN1, R1, R2, TP3, TP4
