File: Hardware/hardware v11/hardware_V11.kicad_sch (KiCad schematic)
At the start: 15 parts, among them U6 STM32G0B1KCUx

Commit message: up
Parts:
- R1: value 510R -> 2.2k
- R2: value 510R -> 1.2k
Changed lines of the file:
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@@
 			)
 		)
-		(property "Value" "510R"
+		(property "Value" "1.2k"
 			(at 48.26 107.95 90)
 			(show_name no)
@@
 			)
 		)
-		(property "Value" "510R"
+		(property "Value" "2.2k"
 			(at 48.26 99.06 90)
 			(show_name no)
