File: Hardware/hardware v11/peripherial.kicad_sch (KiCad schematic)
At the start: 14 parts, among them J1 Micro_SD_Card_Det2

Commit message: up
Parts:
- removed R24: 0R, v9footprintlocal:R_0201_0603Metric_Pad0.64x0.40mm_HandSolder, symbol Device:R_Small
- added C13, C14, C15, C16: 100n, v9footprintlocal:C_0201_0603Metric_Pad0.64x0.40mm_HandSolder, symbol Device:C_Small
- added C24, C25: 4.7u, v9footprintlocal:C_0402_1005Metric, symbol Device:C_Small
- added IC1: DPS368XTSA1, DPS368XTSA1, symbol samacsys:DPS368XTSA1
- added IC2: ICM-42688-P, samacsys:IIM42352, symbol samacsys:ICM-42688-P
- added IC3: MMC5603NJ, samacsys2:MMC5603NJ, symbol samacsys2:MMC5603NJ
- added R22, R23: 4.7k, v9footprintlocal:R_0201_0603Metric_Pad0.64x0.40mm_HandSolder, symbol Device:R_Small
- C21: footprint v9footprintlocal:LED_0402_1005Metric -> v9footprintlocal:C_0402_1005Metric
Connections:
- net 3.3V_AUX: now also C13.1, C14.1, C15.1, C16.1, C24.1, C25.1, IC1.6 (VDDIO), IC1.8 (VDD), IC2.12 (AP_CS), IC2.5 (VDDIO), IC2.8 (VDD), IC3.B1 (VDD), R22.1, R23.2
- net BAT+: now also PA1010D1.9 (VBACKUP)
- net GND: now also C13.2, C14.2, C15.2, C16.2, C24.2, C25.2, IC1.1 (GND_1), IC1.7 (GND_2), IC2.1 (AP_SDO_/_AP_AD0), IC2.10 (RESV_4), IC2.11 (RESV_5), IC2.2 (RESV_1), IC2.3 (RESV_2), IC2.6 (GND), IC2.7 (RESV_3), IC2.9 (INT2_/_FSYNC_/_CLKIN), IC3.A1 (VSA)
- new net SENSOR_SCL: IC1.4 (SCK), IC2.13 (AP_SCL_/_AP_SCLK), IC3.A2 (SCL), R22.2
- new net SENSOR_SDA: IC1.3 (SDI), IC2.14 (AP_SDA_/_AP_SDIO_/_AP_SDI), IC3.B2 (SDA), R23.1
- no-connect marks 7 -> 10
Other:
- note added: "BARO"
- moved on the sheet: C12, R14
