File: Hardware/hardware v11/untitled.kicad_sch (KiCad schematic)
At the start: 21 parts, among them IC1 REG71050DRVR, IC5 LTC4065EDC#TRMPBF, U2 ldln025pu, U3 ldln025pu, U5 ldln025pu

Commit message: up
Parts:
- removed C22, C23: 4.7u, v9footprintlocal:C_0402_1005Metric, symbol Device:C_Small
- removed C9: 0.22u, v9footprintlocal:C_0201_0603Metric_Pad0.64x0.40mm_HandSolder, symbol Device:C
- removed IC1: REG71050DRVR, SON65P200X200X80-7N, symbol samacsys2:REG71050DRVR
- removed R22: 20k, v9footprintlocal:R_0201_0603Metric_Pad0.64x0.40mm_HandSolder, symbol Device:R_Small
Connections:
- net CH_EN is gone; now on net GND: IC5.5 (~{EN})
Other:
- note removed: "A regler pour cutoff"
- moved on the sheet: C4
